File: Hardware/KiCAD/system-testbed/audio-subsystem.kicad_sch (KiCad schematic)
At the start: 20 parts, among them U2 MAX98357A

Commit message: Update-Jumper-Schematic
Parts:
- added J4: Conn_02x13_Odd_Even, symbol Connector_Generic:Conn_02x13_Odd_Even
Connections:
- net +3.3V: now also J4.15 (Pin_15)
- net GND: now also J4.14 (Pin_14), J4.16 (Pin_16), J4.2 (Pin_2)
- new net +5V: J4.18 (Pin_18), J4.20 (Pin_20)
- new net AUDINT_BCLK: J4.3 (Pin_3)
- new net AUDINT_DIN: J4.7 (Pin_7)
- new net AUDINT_LBCLK: J4.5 (Pin_5)
Other:
- note added: "Jumper"
