File: Hardware/KiCAD/system-testbed/power-subsystem.kicad_sch (KiCad schematic)
At the start: 62 parts

Commit message: feat: schematic capture #63
Parts:
- removed H10, H8, H9: MountHole, MountingHole:MountingHole_3.2mm_M3_ISO14580_Pad, symbol Mechanical:MountingHole_Pad
- removed L29: 1uH, Inductor_SMD:L_0603_1608Metric, symbol Device:L
- removed TP29, TP30, TP31, TP32, TP33, TP34, TP35, TP36, TP37, TP38, TP39, TP40, TP41, TP42, TP43, TP44, TP45, TP46, TP47, TP48, TP49: TestPoint, symbol Connector:TestPoint
- added GND1, TP2, TP3, TP4, TP5, TP6, TP7: TestPoint, symbol Connector:TestPoint
- added L4: 1uH, Inductor_SMD:L_0603_1608Metric, symbol Device:L
- H1: value MountHole -> MountingHole_Pad
- U9(Note-checkpinsinsymboleditor)1: renamed from U?; symbol capstone-project:BQ25620RYKR -> 2025-07-10_03-27-55:BQ25620RYKR
- gave numbers to parts that had none: 35
Connections:
- net +BATT is gone; now on net Batt (+): C19.1, R30.2, SW2.3 (C)
- net Batt (+): now also TP4.1; no longer C18.1, U1.C3 (BAT)
- net GND: now also GND1.1
- net SYS: now also L4.2, TP2.1
- net VBUS: now also TP6.1
- net VDD: no longer C16.1, U1.B3 (VDD)
- net Vsys: now also TP3.1
- net at C21.2, R31.1, U9(Note-checkpinsinsymboleditor)1.18 (VBUS): now also TP7.1
- net at R30.1, U9(Note-checkpinsinsymboleditor)1.8 (BAT): now also TP5.1
- net ILIM: no longer names the net of R19.2, U9(Note-checkpinsinsymboleditor)1.4 (ILIM)
- net SW: no longer names the net of C28.1, U9(Note-checkpinsinsymboleditor)1.16 (SW)
- net SW: now also L4.1
- new net: C16.1, U1.B3 (VDD)
- new net Battery(+): C18.1, U1.C3 (BAT)
Other:
- note removed: "Consider having T ponits for these"
- moved on the sheet: BATT1, C16, C18, C19, C20, C21, C22, C24, C28, C33, D1, D2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

Commit message: fix: reannotate and resolve power nets #51
Parts:
- removed GND1, TP2, TP3, TP4, TP5, TP6, TP7: TestPoint, symbol Connector:TestPoint
- removed L4: 1uH, Inductor_SMD:L_0603_1608Metric, symbol Device:L
- added H10, H8, H9: MountHole, MountingHole:MountingHole_3.2mm_M3_ISO14580_Pad, symbol Mechanical:MountingHole_Pad
- added L29: 1uH, Inductor_SMD:L_0603_1608Metric, symbol Device:L
- added TP29, TP30, TP31, TP32, TP33, TP34, TP35, TP36, TP37, TP38, TP39, TP40, TP41, TP42, TP43, TP44, TP45, TP46, TP47, TP48, TP49: TestPoint, symbol Connector:TestPoint
- H1: value MountingHole_Pad -> MountHole
- U?: renamed from U9(Note-checkpinsinsymboleditor)1; symbol 2025-07-10_03-27-55:BQ25620RYKR -> capstone-project:BQ25620RYKR
- renumbered BATT1 to BATT?, C19 to C?, C20 to C?, C16 to C?, C21 to C?, C33 to C?, C22 to C?, C28 to C?, C18 to C?, C24 to C?, D1 to D?, D2 to D?, J to J?, JP7 to JP?, R24 to R?, R21 to R?, R13 to R?, R20 to R?, R28 to R?, R23 to R?, R4 to R?, R26 to R?, R30 to R?, R22 to R?, R19 to R?, R25 to R?, R29 to R?, R31 to R?, R27 to R?, R5 to R?, R15 to R?, SW1 to SW?, SW2 to SW?, TH1 to TH?, U1 to U?
Connections:
- net Battery(+) is gone; now on net Batt (+): C?.1, U?.C3 (BAT)
- net *INT: now also TP36.1
- net *PG: now also TP37.1
- net Batt (+): no longer C?.1, R?.2, SW?.3 (C)
- net GND: now also H10.1, H8.1, H9.1, TP35.1, TP42.1
- net QON: now also TP39.1
- net SCL: now also TP40.1
- net SDA: now also TP41.1
- net STAT: now also TP38.1
- net SYS: now also L29.2, TP33.1, TP48.1
- net TS: now also TP47.1
- net TS_BIAS: now also TP43.1
- net VBUS: now also TP31.1, TP45.1
- net VDD: now also C?.1, U?.B3 (VDD)
- net Vsys: now also TP34.1
- net at C?.2, R?.1, U?.18 (VBUS): now also TP32.1
- net at R?.1, U?.8 (BAT): now also TP30.1
- net SW: now reaches C?.1, U?.16 (SW)
- net SW: now also L29.1, TP44.1
- net ILIM: now reaches R?.2, U?.4 (ILIM)
- net ILIM: now also TP46.1
- new net +BATT: C?.1, R?.2, SW?.3 (C), TP29.1, TP49.1
Other:
- note added: "Consider having T ponits for these"
- moved on the sheet: BATT?, C?, D?, J?, JP?, R?, SW?, TH?, U?
