File: Hardware/KiCAD/system-testbed/power-subsystem.kicad_sch (KiCad schematic)
At the start: 42 parts, among them U5 BQ25620RYKR, U6 BQ24250RGE

Commit message: chore: clear power subsystem schematic, restructure subsheets
Parts:
- removed C14: 10uf, symbol Device:C
- removed C15: 4.7uF, symbol Device:C
- removed C16: 2.2uF, symbol Device:C
- removed C17, C22, C23, C26: 1uF, symbol Device:C
- removed C18: 0.1uF, symbol Device:C
- removed C19: 33nF, symbol Device:C
- removed C20: 47nF, symbol Device:C
- removed C21: 10uF, symbol Device:C
- removed C24: 20uF, symbol Device:C
- removed C25: 22uF, symbol Device:C
- removed D1, D2, D3: LED, symbol Device:LED
- removed L4, L5: 1uH, symbol Device:L
- removed R13, R14, R15, R16, R20, R21, R22, R23, R24, R25, R26, R6: 10k, symbol Device:R
- removed R17, R19, R27, R28, R29, R30, R31: R, symbol Device:R
- removed R18: 1k, symbol Device:R
- removed TH1, TH2: Thermistor_NTC, symbol Device:Thermistor_NTC
- removed U5: BQ25620RYKR, WQFN-HR18__RYK_TEX, symbol 2025-07-10_03-27-55:BQ25620RYKR
- removed U6: BQ24250RGE, BOOSTXL-BATPAKMKII:TI_RGE24, symbol BOOSTXL-BATPAKMKII-eagle-import:BQ24250RGE
Connections:
- no-connect marks 1 -> 0
Other:
- note removed: "BATTERY FEUL GAUGE"
- note removed: "Description of Pins on BQ2425ORGE: > IN - External Power(AC adapter or USB) [Filter IN to PGND with > 2uF Cap] > PMID - (Power Middle) Input power to chargers Buck Converter. (more clarity in connections) > BOOT - High Side MOSFET Gate Driver Supply [Connect a 33nF ceramic Cap (V-rating > 15V) from BOOT to SW to supply the gate drive for the high side MOSFET] > PGND - (Power GND) Ground Terminal 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"
- note removed: "Description of Pins on BQ25620RYKR: > BTST - High Side Switching MOSFET Gate Driver Power Supply [COnnect a 10V or higher rating 47nF cap between SW and BTST as bootstrap cap for driving high side switching MOS] > REGN - Charger Internal Linear Reg o/p: [Connect 10V rating 4.7uF Cap from REGN to PGND] (the REGN LDO o/p is used for internal MOS gate driving voltage and biasing external TS pin ther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"
- note removed: "GPIO-Pins"
- note removed: "HOST"
- note removed: "INPUT/OUTPUT PINS > *PG - indicates if good power source is present. [Connect to pull up rail via 10k res.] -(DIGITAL OUTPUT) > *QON - BATFET Enable or Sys Pow Reset Control i/p: (refer to datasheet for info) -(DIGITAL INPUT) > STAT - o/p reports charging status and any fault conditions. [Connect to pull up rail via 10k res] -(DIGITAL OUTPUT) > *INT - o/p notifies host when a fault occurss or sta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"
- note removed: "I^2C Pins"
- note removed: "Note: STAT Can be connected to Host or REGN for the 3.3V"
- note removed: "Note: STAT, INT and PG can be left floating if un-used"
- note removed: "Pull-Downs"
- note removed: "Pull-Ups"
- note removed: "Relevant Equations: -"
- note removed: "TI-BQ2425ORGE LiPo / Li-Ion Charger"
- note removed: "TI-BQ25620RYK LiPo / Li-Ion BMS (Unit Price: $3.69)"
- note removed: "Temp-Sensor Pin Connection"

Commit message: feat: Power Subsystem Power Supply PCB Fixes #31
Parts:
- added BATT0: M02-JST-2MM-SMT, BOOSTXL-BATPAKMKII:JST-2-SMD, symbol BOOSTXL-BATPAKMKII-eagle-import:M02-JST-2MM-SMT
- added C16: 2.2uF, Capacitor_SMD:C_0201_0603Metric, symbol Device:C
- added C18, C21: 1uF, Capacitor_SMD:C_0201_0603Metric, symbol Device:C
- added C19: 10uf, Capacitor_SMD:C_0201_0603Metric, symbol Device:C
- added C20: 4.7uF, Capacitor_SMD:C_0201_0603Metric, symbol Device:C
- added C22: 0.1uF, Capacitor_SMD:C_0201_0603Metric, symbol Device:C
- added C24: 10uF, Capacitor_SMD:C_0201_0603Metric, symbol Device:C
- added C28: 47nF, Capacitor_SMD:C_0201_0603Metric, symbol Device:C
- added C33: 20uF, Capacitor_SMD:C_0201_0603Metric, symbol Device:C
- added D2, D3: LED, LED_SMD:LED_0201_0603Metric, symbol Device:LED
- added J2: USB_C_Receptacle_USB2.0_14P, Connector_USB:USB_C_Receptacle_GCT_USB4125-xx-x-0190_6P_TopMnt_Horizontal, symbol Connector:USB_C_Receptacle_USB2.0_14P
- added L4: 1uH, Inductor_SMD:L_0201_0603Metric, symbol Device:L
- added R13, R20, R21, R22, R5: 10k, Resistor_SMD:R_0201_0603Metric, symbol Device:R
- added R15 (x2): R, Resistor_SMD:R_0201_0603Metric, symbol Device:R
- added R19 (x2), R20, R4: 5.1k, Resistor_SMD:R_0201_0603Metric, symbol Device:R
- added R23: 1.8M, Resistor_SMD:R_0201_0603Metric, symbol Device:R
- added R24: 0, Resistor_SMD:R_0201_0603Metric, symbol Device:R
- added SW22: SW_SPDT, symbol Switch:SW_SPDT
- added TH2: Thermistor_NTC, symbol Device:Thermistor_NTC
- added U1: BQ25620RYKR, WQFN-HR18__RYK_TEX, symbol 2025-07-10_03-27-55:BQ25620RYKR
- added U5: BQ27427YZFR, DSBGA9-YZF_TEX, symbol 2025-07-20_23-11-47:BQ27427YZFR
Connections:
- new net: C28.1, L4.1, U1.16 (SW)
- new net: BATT0.2, SW22.1 (A), SW22.2 (B)
- new net: C22.2, C24.2, U1.17 (PMID)
- new net: R22.1, R23.1, U5.B1 (BIN)
- new net: D3.2 (A), R13.1
- new net: D2.2 (A), R5.1
- new net: J2.A5 (CC1), R20.2
- new net: C16.1, U5.B3 (VDD)
- new net: R21.2, R24.2, U5.A1 (GPOUT)
- new net: J2.B5 (CC2), R19.2
- new net *INT: R20.1, U1.11 (*INT)
- new net *PG: D3.1 (K), U1.3 (*PG)
- new net +3.3V: R13.2, R19.2, R20.2, R4.2, R5.2
- new net BAT_LOW: R24.1
- new net BTST: C28.2, U1.1 (BTST)
- new net Batt (+): C19.1, SW22.3 (C), U1.8 (BAT)
- new net Battery(+): C18.1, C33.2, L4.2, U1.9 (SYS), U5.C2 (SRX), U5.C3 (BAT)
- new net D-: J2.A7 (D-), J2.B7 (D-), U1.4 (D-)
- new net GND: BATT0.1, C16.2, C18.2, C19.2, C20.1, C21.1, C22.1, C24.1, C33.1, J2.A1 (GND), J2.A12 (GND), J2.A6 (D+), J2.B1 (GND), J2.B12 (GND), J2.B6 (D+), J2.S1 (SHIELD), R15.2, R19.1, R20.1, R22.2, TH2.1, U1.14 (*CE), U1.15 (GND), U1.5 (D+), U5.B2 (VSS), U5.C1 (VSS)
- new net REGN: C20.2, R15.1, U1.2 (REGN)
- new net SCL: R19.1, U1.13 (SCL), U5.A3 (SCL)
- new net SDA: R4.1, U1.12 (SDA), U5.A2 (SDA)
- new net STAT: D2.1 (K), U1.10 (STAT)
- new net TS: R15.1, R15.2, TH2.2, U1.6 (TS)
- new net VBUS: C21.2, J2.A4 (VBUS), J2.A9 (VBUS), J2.B4 (VBUS), J2.B9 (VBUS), U1.18 (VBUS)
- new net VDD: R21.1, R23.2
- no-connect marks 0 -> 1
Other:
- note added: "Batt Charger (BMS)"
- note added: "Battery Connection"
- note added: "Charge Connector"
- note added: "Connection to ESP32"
- note added: "Fuel Gauge"
- note added: "GPIO connection"
- note added: "GPIO-Pins"
- note added: "I^2C Pins"
- note added: "Temp-Sensor Pin Connection"
- note added: "To BMS 'SYS'"
- note added: "When Battery is attatched it pulls low"
- note added: "enables standard usb power."
- note added: "verifies BIN HIGH when battery removed"

Commit message: feat: Update to PSU Power Supply PCB Fixes #31
Parts:
- removed D3: LED, LED_SMD:LED_0201_0603Metric, symbol Device:LED
- removed R13, R5: 10k, Resistor_SMD:R_0201_0603Metric, symbol Device:R
- removed R15 (x2): R, Resistor_SMD:R_0201_0603Metric, symbol Device:R
- removed R4: 5.1k, Resistor_SMD:R_0201_0603Metric, symbol Device:R
- removed TH2: Thermistor_NTC, symbol Device:Thermistor_NTC
- removed U1: BQ25620RYKR, WQFN-HR18__RYK_TEX, symbol 2025-07-10_03-27-55:BQ25620RYKR
- added D1: LED, LED_SMD:LED_0201_0603Metric, symbol Device:LED
- added JP7: SolderJumper_3_Bridged12, symbol Jumper:SolderJumper_3_Bridged12
- added R21, R22, R23, R24: 10k, Resistor_SMD:R_0201_0603Metric, symbol Device:R
- added R25, R26: R, Resistor_SMD:R_0201_0603Metric, symbol Device:R
- added SW1: SW_Push, symbol Switch:SW_Push
- added TH1: Thermistor_NTC, symbol Device:Thermistor_NTC
- added U9(Note-checkpinsinsymboleditor)1: BQ25622RYKR, capstone-project:WQFN-HR18__RYK_TEX, symbol 2025-07-10_03-27-55:BQ25620RYKR
- R19: value 5.1k -> TBD
- U1: renamed from U5; footprint DSBGA9-YZF_TEX -> capstone-project:DSBGA9-YZF_TEX
- renumbered BATT0 to BATT1, J2 to J1, R22 to R13, R21 to R15, R19 to R27, R20 to R28, R24 to R4, R23 to R5, SW22 to SW2
Connections:
- net *INT: now also R24.1, U9(Note-checkpinsinsymboleditor)1.11 (*INT); no longer R20.1
- net *PG: now also D2.1 (K), U9(Note-checkpinsinsymboleditor)1.3 (PG)
- net +3.3V: now also R21.2, R22.2, R23.2, R24.2; no longer R19.2
- net BTST: now also U9(Note-checkpinsinsymboleditor)1.1 (BTST)
- net Batt (+): now also U9(Note-checkpinsinsymboleditor)1.8 (BAT)
- net Battery(+): no longer C33.2, L4.2, U1.C2 (SRX)
- net GND: now also R19.1, R26.2, SW1.2, TH1.1, U9(Note-checkpinsinsymboleditor)1.14 (*CE), U9(Note-checkpinsinsymboleditor)1.15 (GND); no longer J1.A6 (D+), J1.B6 (D+), R13.2
- net SCL: now also R21.1, U9(Note-checkpinsinsymboleditor)1.13 (SCL); no longer R19.1
- net SDA: now also R20.1, U9(Note-checkpinsinsymboleditor)1.12 (SDA)
- net STAT: now also D1.1 (K), U9(Note-checkpinsinsymboleditor)1.10 (STAT); no longer D2.1 (K)
- net TS: now also R25.2, R26.1, TH1.2, U9(Note-checkpinsinsymboleditor)1.6 (TS)
- net VBUS: now also U9(Note-checkpinsinsymboleditor)1.18 (VBUS)
- net at C28.1, L4.1: now also U9(Note-checkpinsinsymboleditor)1.16 (SW)
- net at C22.2, C24.2: now also U9(Note-checkpinsinsymboleditor)1.17 (PMID)
- net at D2.2 (A): now also R23.1
- net D-: no longer names the net of J1.A7 (D-)
- net D-: no longer J1.B7 (D-)
- net REGN: no longer names the net of C20.2
- net REGN: now also U9(Note-checkpinsinsymboleditor)1.2 (REGN)
- new net: D1.2 (A), R22.1
- new net: R19.2, U9(Note-checkpinsinsymboleditor)1.4 (ILIM)
- new net QON: SW1.1, U9(Note-checkpinsinsymboleditor)1.7 (QON)
- new net TS_BIAS: R25.1, U9(Note-checkpinsinsymboleditor)1.5 (TS_BIAS)
- new net VSS: R13.2
- new net Vsys: C33.2, L4.2, U1.C2 (SRX), U9(Note-checkpinsinsymboleditor)1.9 (SYS)
- no-connect marks 1 -> 7
Other:
- note added: "Verfy connection of BIN pin"
- moved on the sheet: R27, R28

Commit message: fix: add power devices to library
Parts:
- added GND, TP2, TP3, TP4, TP5, TP6, TP7: TestPoint, symbol Connector:TestPoint
- added H1: MountingHole_Pad, MountingHole:MountingHole_3.2mm_M3_ISO14580_Pad, symbol Mechanical:MountingHole_Pad
- added R29, R30, R31: 0, Resistor_SMD:R_0603_1608Metric, symbol Device:R
- C16, C18, C19, C20, C21, C22, C24, C28, C33: footprint Capacitor_SMD:C_0201_0603Metric -> Capacitor_SMD:C_0603_1608Metric
- L4: footprint Inductor_SMD:L_0201_0603Metric -> Inductor_SMD:L_0603_1608Metric
- R13, R15, R19, R20, R21, R22, R23, R24, R25, R26, R27, R28, R4, R5: footprint Resistor_SMD:R_0201_0603Metric -> Resistor_SMD:R_0603_1608Metric
Connections:
- net Batt (+): now also R30.2, TP4.1; no longer U9(Note-checkpinsinsymboleditor)1.8 (BAT)
- net GND: now also GND.1, H1.1
- net VBUS: now also R31.2, TP6.1; no longer C21.2, U9(Note-checkpinsinsymboleditor)1.18 (VBUS)
- net Vsys: now also R29.1, TP3.1; no longer C33.2, L4.2, U1.C2 (SRX), U9(Note-checkpinsinsymboleditor)1.9 (SYS)
- new net: C21.2, R31.1, TP7.1, U9(Note-checkpinsinsymboleditor)1.18 (VBUS)
- new net: R30.1, TP5.1, U9(Note-checkpinsinsymboleditor)1.8 (BAT)
- new net SYS: C33.2, L4.2, R29.2, TP2.1, U1.C2 (SRX), U9(Note-checkpinsinsymboleditor)1.9 (SYS)
Other:
- note added: "Mounting Holes"
- note added: "Test Points"
- moved on the sheet: BATT1, C16, C18, C19, C20, C21, C22, C24, C28, C33, D1, D2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

Commit message: fix: correct input and output for labels #51
Parts:
- renumbered GND to GND1, J1 to J
Changed lines of the file:
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@@
 	)
 	(hierarchical_label "SCL"
-		(shape bidirectional)
+		(shape input)
 		(at 207.01 116.84 0)
 		(effects
@@
 		(dnp no)
 		(fields_autoplaced yes)
-		(property "Reference" "GND"
+		(property "Reference" "GND1"
 			(at 331.47 136.3979 0)
 			(effects
@@
 			(project ""
 				(path "/72756aea-0ff9-4757-9699-8d0f18588f6f/9fe85a84-eb88-4cb0-ad9c-c856ce023e7b"
-					(reference "GND")
+					(reference "GND1")
 					(unit 1)
 				)
@@
 		(on_board yes)
 		(dnp no)
-		(property "Reference" "J1"
+		(property "Reference" "J"
 			(at 404.114 37.846 0)
 			(effects
@@
 			(project "system-testbed"
 				(path "/72756aea-0ff9-4757-9699-8d0f18588f6f/9fe85a84-eb88-4cb0-ad9c-c856ce023e7b"
-					(reference "J1")
+					(reference "J")
 					(unit 1)
 				)
@@
 		(dnp no)
 		(fields_autoplaced yes)
-		(property "Reference" "#PWR013"
+		(property "Reference" "#PWR0135"
 			(at 101.6 77.47 0)
 			(effects
@@
 			(project "system-testbed"
 				(path "/72756aea-0ff9-4757-9699-8d0f18588f6f/9fe85a84-eb88-4cb0-ad9c-c856ce023e7b"
-					(reference "#PWR013")
-					(unit 1)
-				)
+					(reference "#PWR0135")
+					(unit 1)
+				)

Commit message: fix: Cleaned up structure of BMS PSU Schematic Capture Fixes #51
Parts:
- removed C33: 20uF, Capacitor_SMD:C_0603_1608Metric, symbol Device:C
- removed JP7: SolderJumper_3_Bridged12, symbol Jumper:SolderJumper_3_Bridged12
- removed R31: 0, Resistor_SMD:R_0603_1608Metric, symbol Device:R
- removed TP6, TP7: TestPoint, symbol Connector:TestPoint
- added C73: 4.7uF, Capacitor_SMD:C_0603_1608Metric, symbol Device:C
- added H10, H8, H9: MountHole, MountingHole:MountingHole_3.2mm_M3_ISO14580_Pad, symbol Mechanical:MountingHole_Pad
- added R38: 0, Resistor_SMD:R_0603_1608Metric, symbol Device:R
- added TP30, TP31, TP32, TP33, TP37, TP38, TP40, TP41, TP43, TP44, TP45: TestPoint, symbol Connector:TestPoint
- C20: value 4.7uF -> 1uF
- C21: value 1uF -> 47nF
- C28: value 47nF -> 20uF
- H1: value MountingHole_Pad -> MountHole
- U7: renamed from U9(Note-checkpinsinsymboleditor)1; symbol 2025-07-10_03-27-55:BQ25620RYKR -> capstone-project:BQ25620RYKR
- renumbered J to J6, R5 to R13, R13 to R15, R15 to R19, R30 to R20, R19 to R21, R20 to R22, R21 to R23, R22 to R25, R23 to R26, R24 to R27, R25 to R28, R26 to R29, R29 to R30, R27 to R31, R28 to R37, R4 to R5, SW1 to SW2, SW2 to SW6, TP4 to TP2, GND1 to TP29, TP5 to TP3, TP2 to TP6, TP3 to TP7
Connections:
- net Battery(+) is gone; now on net +BATT: C18.1, U1.C3 (BAT)
- net SYS is gone; now on net SRX: L4.2, R30.2, TP6.1, U1.C2 (SRX), U7.9 (SYS)
- net VSS is gone; now on net GND: R15.2
- net *INT: now also TP30.1
- net *PG: now also TP31.1
- net +3.3V: now also R19.1
- net GND: now also C28.1, C73.1, H10.1, H8.1, H9.1; no longer C21.1
- net STAT: now also TP32.1
- net TS: now also TP41.1
- net TS_BIAS: now also TP37.1
- net VBUS: now also R38.1, TP45.1
- net VDD: no longer R19.1
- net at C20.2: now also U7.18 (VBUS), R38.2, TP44.1; no longer U7.2 (REGN)
- net at C21.2: now also U7.1 (BTST); no longer U7.18 (VBUS)
- net T_SW: now reaches L4.1, U7.16 (SW)
- net T_SW: now also C21.1, TP38.1; no longer C28.1
- net ILIM: now reaches R21.2, U7.4 (ILIM)
- net ILIM: now also TP40.1
- net BTST renamed SRX
- net SRX: no longer U7.1 (BTST)
- net Batt (+) renamed +BATT
- net +BATT: now also TP43.1
- net QON renamed *QON
- net *QON: now also TP33.1
- new net: C73.2, U7.2 (REGN)
- no-connect marks 7 -> 4
Other:
- note added: "VDD is LDO output of approx 1.8V"
- note removed: "GPIO connection"
- note removed: "To BMS 'SYS'"
- note removed: "Verfy connection of BIN pin"
- moved on the sheet: BATT1, C16, C18, C19, C22, C24, D1, D2, H1, J6, R13, R15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

Commit message: fix: fixing labels PSU Schematic Capture Fixes #51
Parts:
- added R24: 0, Resistor_SMD:R_0603_1608Metric, symbol Device:R
Connections:
- net *PG: no longer TP31.1
- net GND: now also R24.1; no longer C73.1, U7.15 (GND)
- net STAT: no longer TP32.1
- net VDD: now also C16.1, U1.B3 (VDD)
- net Vsys renamed Vout
- new net PGND: C73.1, R24.2, U7.15 (GND)
Other:
- note added: "Note: resistor in series with power input conflicts with ERC to not see Power output going in. (Reason for numerious power flags)"
- moved on the sheet: C18

Commit message: Feat: Add Regulators & Power distribution Schematics, and new power IC libraries
Parts:
- added C301: 4.7u, symbol Device:C
- added C302, C303, C304, C307: 1.0u, symbol Device:C
- added C310: 100n, symbol Device:C
- added D301: ESDA25W, capstone-project:SOT65P210X110-3N, symbol capstone-project:ESDA25W
- added D302, D303: ESDA25P35-1U1M, capstone-project:TVS_ESDA25P35-1U1M, symbol capstone-project:ESDA25P35-1U1M
- added D305: ESDA25P35-1U1M, ESDA25P35-1U1M:TVS_ESDA25P35-1U1M, symbol capstone-project:ESDA25P35-1U1M
- added J301: 217177-0001, capstone-project:2171770001, symbol capstone-project:217177-0001
- added LED301: LTST-C190KRKT, capstone-project:LTST-C190KRKT, symbol LTST-C190KRKT:LTST-C190KRKT
- added Q301: 2N7002, Package_TO_SOT_SMD:SOT-23, symbol Transistor_FET:2N7002
- added Q302, Q303: STL6P3LLH6, capstone-project:TRANS_STL6P3LLH6, symbol capstone-project:STL6P3LLH6
- added R301: 330, symbol Device:R
- added R306, R307, R312, R_pullup301: 10k, symbol Device:R
- added R308, R309, R316: 100k, symbol Device:R
- added R310: 5.1k, symbol Device:R
- added R311: 2.5k, symbol Device:R
- added R313: 470, symbol Device:R
- added R314, R320, R_gate301: 1k, symbol Device:R
- added R315: 22k, symbol Device:R
- added R321: 100, symbol Device:R
- added U301: STUSB4500QTR, capstone-project:STUSB4500QTR, symbol capstone-project:STUSB4500QTR
- added U303: TPS25200DRVR, capstone-project:TPS25200DRVR, symbol capstone-project:TPS25200DRVR
- renumbered BATT1 to BATT301, C16 to C305, C18 to C306, C19 to C308, C73 to C309, C21 to C311, C22 to C312, C24 to C313, C20 to C314, C28 to C315, D1 to D304, D2 to D306, H1 to H301, H8 to H302, H9 to H303, H10 to H304, J6 to J302, L4 to L301, R5 to R302, R13 to R303, R15 to R304, R19 to R305, R24 to R317, R20 to R318, R21 to R319, R22 to R322, R23 to R323, R25 to R324, R26 to R325, R27 to R326, R28 to R327, R29 to R328, R38 to R329, R30 to R330, R31 to R331, R37 to R332, SW2 to SW301, SW6 to SW302, TH1 to TH301, TP2 to TP301, TP3 to TP302, TP6 to TP303, TP44 to TP304, TP45 to TP305, TP7 to TP306, TP29 to TP307, TP30 to TP308, TP31 to TP309, TP32 to TP310, TP33 to TP311, TP43 to TP312, TP37 to TP313, TP38 to TP314, TP40 to TP315, TP41 to TP316, U1 to U302, U7 to U304
Connections:
- net GND: now also C301.2, C302.1, C303.1, C304.1, C307.2, D301.3, D302.A, D305.A, J301.C1 (GND_1), J301.C6 (GND_2), J301.MH1, J301.MH2, J301.MH3, J301.MH4, Q301.2 (S), R308.1, R309.1, R310.1, R311.1, R312.1, U301.10 (GND), U301.22 (VSYS), U303.5 (GND), U303.7 (EP)
- net SCL: now also U301.7 (SCL)
- net SDA: now also U301.8 (SDA)
- new net: Q301.3 (D), R_pullup301.2
- new net: Q302.1, Q302.2, Q302.3, Q303.1, Q303.2, Q303.3, R316.2
- new net: Q302.4, Q303.4, R315.2, R316.1, R321.2
- new net: D303.A, Q302.5_8, R313.2, U303.1 (OUT)
- new net: R306.1, R308.2, R309.2, U301.12 (ADDR0)
- new net: Q301.1 (G), R_gate301.1
- new net: LED301.1 (K), R301.1
- new net: R311.2, U303.2 (ILIM)
- new net: R315.1, R_gate301.2, U301.16 (VBUS_EN_SNK)
- new net: C307.1, D303.C, R313.1, R314.2
- new net: R307.1, U301.13 (ADDR1)
- new net: C310.1, R321.1
- new net: R312.2, U301.6 (RESET)
- new net: R320.2, U301.9 (DISCH)
- new net 2V7: C302.2, C303.2, C304.2, R306.2, R307.2, U301.21 (VREG_1V2), U301.23 (VREG_2V7), U301.24 (VDD)
- new net USB_CC1: D301.2, J301.C3 (CC1), R310.2, U301.1 (CC1DB), U301.2 (CC1)
- new net USB_CC2: D301.1, J301.C4 (CC2), U301.4 (CC2), U301.5 (CC2DB)
- new net USB_VBUS: C301.1, D302.C, J301.C2 (VBUS_1), J301.C5 (VBUS_2), U303.6 (IN)
- new net VBUS_VS_DISCH: R314.1, U301.18 (VBUS_VS_DISCH)
- new net Vout_3.3 V: LED301.2 (A)
- new net Vsink: C310.2, D305.C, Q303.5_8, R320.1
- new net eFUSE_EN: R_pullup301.1, U303.4 (EN)
- new net eFUSE_FAULT: R301.2, U303.3 (~{FAULT})
- no-connect marks 4 -> 10
Other:
- added sheet Other_Blocks (Other Blocks.kicad_sch)
- note added: "E: Control Plane (Firmware & MCU)"
