File: Hardware/KiCAD/system-testbed/power-subsystem.kicad_sch (KiCad schematic)
At the start: 90 parts, among them J301 217177-0001, J302 USB_C_Receptacle_USB2.0_14P, Q301 2N7002, Q302 STL6P3LLH6, Q303 STL6P3LLH6, SW301 SW_Push, SW302 SW_SPDT, U301 STUSB4500QTR, U302 BQ27427YZFR, U303 TPS25200DRVR, U304 BQ25622RYKR

Commit message: Fix: Changed IC positions
Parts:
- removed R310: 5.1k, symbol Device:R
- added R?: 5.1k, symbol Device:R
- renumbered BATT301 to BATT401, C305 to C405, C306 to C406, C308 to C408, C309 to C409, C311 to C411, C312 to C412, C313 to C413, C314 to C414, C315 to C415, C302 to C?, C303 to C?, C301 to C?, C310 to C?, C307 to C?, C304 to C?, D304 to D404, D306 to D406, D302 to D?, D301 to D?, D305 to D?, D303 to D?, H301 to H401, H302 to H402, H303 to H403, H304 to H404, J301 to J401, J302 to J402, L301 to L401, LED301 to LED401, Q302 to Q?, Q301 to Q?, Q303 to Q?, R301 to R401, R302 to R402, R303 to R403, R304 to R404, R305 to R405, R315 to R415, R317 to R417, R318 to R418, R319 to R419, R322 to R422, R323 to R423, R324 to R424, R325 to R425, R326 to R426, R327 to R427, R328 to R428, R329 to R429, R330 to R430, R331 to R431, R332 to R432, R308 to R?, R316 to R?, R306 to R?, R311 to R?, R314 to R?, R307 to R?, R321 to R?, R313 to R?, R312 to R?, R309 to R?, R320 to R?, R_gate301 to R_gate?, R_pullup301 to R_pullup?, SW301 to SW401, SW302 to SW402, TH301 to TH401, TP301 to TP401, TP302 to TP402, TP303 to TP403, TP304 to TP404, TP305 to TP405, TP306 to TP406, TP307 to TP407, TP308 to TP408, TP309 to TP409, TP310 to TP410, TP311 to TP411, TP312 to TP412, TP313 to TP413, TP314 to TP414, TP315 to TP415, TP316 to TP416, U302 to U402, U303 to U403, U304 to U404, U301 to U?
Connections:
- net GND: now also R?.2; no longer U?.10 (GND)
- net USB_CC1: now also R?.1
Other:
- note removed: "E: Control Plane (Firmware & MCU)"
- moved on the sheet: C?, D?, LED401, Q?, R401, R415, R?, R_gate?, R_pullup?, U403, U?

Commit message: Feat: Added footprint for TVS Diode
Parts:
- D?: footprint ESDA25P35-1U1M:TVS_ESDA25P35-1U1M -> capstone-project:TVS_ESDA25P35-1U1M
Changed lines of the file:
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@@
 			)
 		)
-		(property "Footprint" "ESDA25P35-1U1M:TVS_ESDA25P35-1U1M"
+		(property "Footprint" "capstone-project:TVS_ESDA25P35-1U1M"
 			(at 308.61 146.05 0)
 			(effects

Commit message: fix: allow for DRC use in PCB editor by successful reannotation
Parts:
- removed C405: 2.2uF, Capacitor_SMD:C_0603_1608Metric, symbol Device:C
- removed C406, C414: 1uF, Capacitor_SMD:C_0603_1608Metric, symbol Device:C
- removed C408: 10uf, Capacitor_SMD:C_0603_1608Metric, symbol Device:C
- removed C409: 4.7uF, Capacitor_SMD:C_0603_1608Metric, symbol Device:C
- removed C411: 47nF, Capacitor_SMD:C_0603_1608Metric, symbol Device:C
- removed C412: 0.1uF, Capacitor_SMD:C_0603_1608Metric, symbol Device:C
- removed C413: 10uF, Capacitor_SMD:C_0603_1608Metric, symbol Device:C
- removed C415: 20uF, Capacitor_SMD:C_0603_1608Metric, symbol Device:C
- removed C? (x3): 1.0u, symbol Device:C
- removed C?: 4.7u, symbol Device:C
- removed C?: 100n, symbol Device:C
- removed D404, D406: LED, LED_SMD:LED_0201_0603Metric, symbol Device:LED
- removed D? (x2): ESDA25P35-1U1M, capstone-project:TVS_ESDA25P35-1U1M, symbol capstone-project:ESDA25P35-1U1M
- removed H401, H402, H403, H404: MountHole, MountingHole:MountingHole_3.2mm_M3_ISO14580_Pad, symbol Mechanical:MountingHole_Pad
- removed J401: 217177-0001, capstone-project:2171770001, symbol capstone-project:217177-0001
- removed J402: USB_C_Receptacle_USB2.0_14P, Connector_USB:USB_C_Receptacle_GCT_USB4125-xx-x-0190_6P_TopMnt_Horizontal, symbol Connector:USB_C_Receptacle_USB2.0_14P
- removed L401: 1uH, Inductor_SMD:L_0603_1608Metric, symbol Device:L
- removed LED401: LTST-C190KRKT, capstone-project:LTST-C190KRKT, symbol LTST-C190KRKT:LTST-C190KRKT
- removed Q?: 2N7002, Package_TO_SOT_SMD:SOT-23, symbol Transistor_FET:2N7002
- removed Q?: STL6P3LLH6, capstone-project:TRANS_STL6P3LLH6, symbol capstone-project:STL6P3LLH6
- removed R402, R417, R418, R429, R430: 0, Resistor_SMD:R_0603_1608Metric, symbol Device:R
- removed R403: 1.8M, Resistor_SMD:R_0603_1608Metric, symbol Device:R
- removed R404, R405, R422, R423, R424, R425, R426: 10k, Resistor_SMD:R_0603_1608Metric, symbol Device:R
- removed R419: TBD, Resistor_SMD:R_0603_1608Metric, symbol Device:R
- removed R427, R428: R, Resistor_SMD:R_0603_1608Metric, symbol Device:R
- removed R431, R432: 5.1k, Resistor_SMD:R_0603_1608Metric, symbol Device:R
- removed R?: 5.1k, symbol Device:R
- removed R? (x2): 100k, symbol Device:R
- removed R? (x3), R_pullup?: 10k, symbol Device:R
- removed R?: 2.5k, symbol Device:R
- removed R?: 100, symbol Device:R
- removed R?: 1k, symbol Device:R
- removed SW401: SW_Push, symbol Switch:SW_Push
- removed SW402: SW_SPDT, symbol Switch:SW_SPDT
- removed TH401: Thermistor_NTC, symbol Device:Thermistor_NTC
- removed TP401, TP402, TP403, TP404, TP405, TP406, TP407, TP408, TP409, TP410, TP411, TP412, TP413, TP414, TP415, TP416: TestPoint, symbol Connector:TestPoint
- removed U402: BQ27427YZFR, capstone-project:DSBGA9-YZF_TEX, symbol 2025-07-20_23-11-47:BQ27427YZFR
- removed U403: TPS25200DRVR, capstone-project:TPS25200DRVR, symbol capstone-project:TPS25200DRVR
- removed U404: BQ25622RYKR, capstone-project:WQFN-HR18__RYK_TEX, symbol capstone-project:BQ25620RYKR
- added C135: 2.2uF, Capacitor_SMD:C_0603_1608Metric, symbol Device:C
- added C136, C147, C149: 1uF, Capacitor_SMD:C_0603_1608Metric, symbol Device:C
- added C137, C139, C140: 1.0u, symbol Device:C
- added C141: 10uf, Capacitor_SMD:C_0603_1608Metric, symbol Device:C
- added C142: 4.7uF, Capacitor_SMD:C_0603_1608Metric, symbol Device:C
- added C143: 100n, symbol Device:C
- added C144: 47nF, Capacitor_SMD:C_0603_1608Metric, symbol Device:C
- added C145: 0.1uF, Capacitor_SMD:C_0603_1608Metric, symbol Device:C
- added C146: 10uF, Capacitor_SMD:C_0603_1608Metric, symbol Device:C
- added C148: 20uF, Capacitor_SMD:C_0603_1608Metric, symbol Device:C
- added C150: 4.7u, symbol Device:C
- added D10, D9: ESDA25P35-1U1M, capstone-project:TVS_ESDA25P35-1U1M, symbol capstone-project:ESDA25P35-1U1M
- added D7, D8: LED, LED_SMD:LED_0603_1608Metric, symbol Device:LED
- added J5: 217177-0001, capstone-project:2171770001, symbol capstone-project:217177-0001
- added L41: 1uH, Inductor_SMD:L_0603_1608Metric, symbol Device:L
- added LED1: LTST-C190KRKT, capstone-project:LTST-C190KRKT, symbol LTST-C190KRKT:LTST-C190KRKT
- added Q4: NMOS, symbol Simulation_SPICE:NMOS
- added Q5: 2N7002, Package_TO_SOT_SMD:SOT-23, symbol Transistor_FET:2N7002
- added Q7: STL6P3LLH6, capstone-project:TRANS_STL6P3LLH6, symbol capstone-project:STL6P3LLH6
- added R48: 1.8M, Resistor_SMD:R_0603_1608Metric, symbol Device:R
- added R49: bias, Resistor_SMD:R_0603_1608Metric, symbol Device:R
- added R50, R51, R52, R63, R65, R68, R69, R70: 10k, Resistor_SMD:R_0603_1608Metric, symbol Device:R
- added R53, R54, R58, R_pullup2: 10k, symbol Device:R
- added R55, R56: 100k, symbol Device:R
- added R57, R73, R74: 0, Resistor_SMD:R_0603_1608Metric, symbol Device:R
- added R61: TBD, Resistor_SMD:R_0603_1608Metric, symbol Device:R
- added R66: 1k, symbol Device:R
- added R67: 100, symbol Device:R
- added R71, R72: R, Resistor_SMD:R_0603_1608Metric, symbol Device:R
- added R75: 5.1k, symbol Device:R
- added R76: 2.5k, symbol Device:R
- added S1: 100SP1T1B4M2QE, capstone-project:SW_100SP1T1B4M2QE, symbol capstone-project:100SP1T1B4M2QE
- added SW6: SW_Push, symbol Switch:SW_Push
- added TH1: Thermistor_NTC, Resistor_THT:R_Axial_DIN0204_L3.6mm_D1.6mm_P2.54mm_Vertical, symbol Device:Thermistor_NTC
- added TP29, TP30, TP31, TP32, TP33, TP34: TestPoint, symbol Connector:TestPoint
- added TP35, TP36, TP37, TP38, TP39, TP40, TP41, TP42, TP43: TestPoint, TestPoint:TestPoint_Loop_D2.60mm_Drill1.6mm_Beaded, symbol Connector:TestPoint
- added U16: BQ27427YZFR, capstone-project:DSBGA9-YZF_TEX, symbol 2025-07-20_23-11-47:BQ27427YZFR
- added U17: BQ25622RYKR, capstone-project:WQFN-HR18__RYK_TEX, symbol capstone-project:BQ25620RYKR
- added U18: TPS25200DRVR, capstone-project:TPS25200DRVR, symbol capstone-project:TPS25200DRVR
- BATT1: renamed from BATT401; footprint BOOSTXL-BATPAKMKII:JST-2-SMD -> Connector_JST:JST_GH_BM02B-GHS-TBT_1x02-1MP_P1.25mm_Vertical
- gave numbers to parts that had none: 9
- renumbered R401 to R47, R415 to R62
Connections:
- net *INT: now also R70.1, TP36.1, U17.11 (*INT)
- net *PG: now also D8.1 (K), TP38.1, U17.3 (*PG)
- net *QON: now also SW6.1, U17.7 (*QON)
- net +3.3V: now also R51.1, R63.2, R65.2, R68.2, R69.2, R70.2
- net +BATT: now also C136.1, C141.1, S1.3, TP29.1, TP30.1, TP39.1, U16.C3 (BAT), U17.8 (BAT)
- net 2V7: now also C137.2, C139.2, R53.2, R54.2
- net BAT_LOW: now also R51.2, U16.A1 (GPOUT)
- net GND: now also C135.2, C136.2, C137.1, C139.1, C140.2, C141.2, C145.1, C146.1, C147.1, C148.1, C149.1, C150.2, D10.A, D9.A, J5.C1 (GND_1), J5.C6 (GND_2), J5.MH1, J5.MH2, J5.MH3, J5.MH4, Q4.3 (S), Q5.2 (S), R50.1, R50.2, R55.1, R56.1, R57.1, R58.1, R61.1, R72.2, R75.2, R76.1, SW6.2, TH1.1, TP35.1, U16.B2 (VSS), U16.C1 (VSS), U17.14 (*CE), U18.5 (GND), U18.7 (EP)
- net ILIM: now also R61.2, TP42.1, U17.4 (ILIM)
- net PGND: now also C142.1, R57.2, U17.15 (GND)
- net SCL: now also R65.1, U16.A3 (SCL), U17.13 (SCL)
- net SDA: now also R63.1, U16.A2 (SDA), U17.12 (SDA)
- net SRX: now also C148.2, C149.2, L41.2, R74.2, TP32.1, U16.C2 (SRX), U17.9 (SYS)
- net STAT: now also D7.1 (K), TP37.1, U17.10 (STAT)
- net TS: now also R71.2, R72.1, TH1.2, TP43.1, U17.6 (TS)
- net TS_BIAS: now also R71.1, TP40.1, U17.5 (TS_BIAS)
- net T_SW: now also C144.1, L41.1, TP41.1, U17.16 (SW)
- net USB_CC1: now also J5.C3 (CC1), R75.1
- net USB_CC2: now also J5.C4 (CC2)
- net VBUS: now also C150.1, D10.C, J5.C2 (VBUS_1), J5.C5 (VBUS_2), R73.1, TP33.1, U18.6 (IN)
- net VDD: now also C135.1, R48.2, U16.B3 (VDD)
- net Vout: now also R74.1, TP34.1
- net Vout_3.3 V: now also LED1.2 (A)
- net Vsink: now also C143.2, D9.C, Q7.5_8, R66.1
- net eFUSE_EN: now also R_pullup2.1, U18.4 (EN)
- net eFUSE_FAULT: now also U18.3 (~{FAULT})
- net at BATT1.2: now also S1.1, S1.2
- net at Q6.1, Q6.2, Q6.3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: now also Q7.1, Q7.2, Q7.3
- net at Q6.4, R62.2, R64.1: now also Q7.4, R67.2
- net Breaker: now reaches D6.A, Q6.5_8, R59.2
- net Breaker: now also U18.1 (OUT)
- net at U15.12 (ADDR0): now also R53.1, R55.2, R56.2
- net at R_gate2.1: now also Q5.1 (G)
- net at R47.1: now also LED1.1 (K)
- net at D6.C, R59.1, R60.2: now also C140.1
- net at U15.13 (ADDR1): now also R54.1
- net at U15.6 (RESET): now also R58.2
- net at U15.9 (DISCH): now also R66.2
- new net: Q4.1 (D), R52.1
- new net: Q4.2 (G), R49.2
- new net: C143.1, R67.1
- new net: C147.2, R73.2, TP31.1, U17.18 (VBUS)
- new net: R48.1, U16.B1 (BIN)
- new net: C144.2, U17.1 (BTST)
- new net: C145.2, C146.2, U17.17 (PMID)
- new net: C142.2, U17.2 (REGN)
- new net: D8.2 (A), R69.1
- new net: Q5.3 (D), R_pullup2.2
- new net: R76.2, U18.2 (ILIM)
- new net: D7.2 (A), R68.1
- new net BIN: R52.2
- no-connect marks 10 -> 6
Other:
- removed sheet Other_Blocks
- note removed: "When Battery is attatched it pulls low"
- note removed: "enables standard usb power."
- note removed: "verifies BIN HIGH when battery removed"
- moved on the sheet: BATT1, C138, D5, D6, Q6, R47, R59, R60, R62, R64, R_gate2, U15
