File: Hardware/KiCAD/system-testbed/Other Blocks.kicad_sch (KiCad schematic)
At the start: 59 parts, among them U305 TPS63020QDSJRQ1, U306 TPS61088RHLR, U307 TPS7A90, U308 TPS22916BYFPR, U309 TPS22916BYFPR, U310 TPS22965DSGR

Commit message: Fix: Changed IC positions
Parts:
- C?: renamed from C346; value 0.1 -> 0.1u
- renumbered C318 to C?, C348 to C?, C326 to C?, C327 to C?, C339 to C?, C320 to C?, C343 to C?, C335 to C?, C332 to C?, C337 to C?, C344 to C?, C336 to C?, C325 to C?, C341 to C?, C321 to C?, C323 to C?, C324 to C?, C347 to C?, C328 to C?, C316 to C?, C338 to C?, C319 to C?, C340 to C?, C331 to C?, C317 to C?, C329 to C?, C333 to C?, C334 to C?, C322 to C?, C330 to C?, C345 to C?, C342 to C?, L303 to L?, L302 to L?, R337 to R?, R340 to R?, R338 to R?, R339 to R?, R342 to R?, R336 to R?, R334 to R?, R343 to R?, R341 to R?, R335 to R?, R333 to R?, R344 to R?, TP318 to TP?, TP322 to TP?, TP320 to TP?, TP319 to TP?, TP321 to TP?, TP317 to TP?, U310 to U?, U306 to U?, U307 to U?, U309 to U?, U308 to U?, U305 to U?
Other:
- note removed: "C: DC-DC Conversion (Voltage Regulation)"
- moved on the sheet: C?

Commit message: fix: allow for DRC use in PCB editor by successful reannotation
Parts:
- C100: renamed from C?; value 10u -> 10uF; footprint (none) -> Capacitor_SMD:C_0402_1005Metric
- C101: renamed from C?; value 0.1u -> 1uF; footprint (none) -> Capacitor_SMD:C_0402_1005Metric
- C102: renamed from C?; value 10u -> 20uF; footprint (none) -> Capacitor_SMD:C_0402_1005Metric
- C103: renamed from C?; value 2.2u -> C; footprint (none) -> Capacitor_SMD:C_0402_1005Metric
- C104: renamed from C?; value 0.1u -> C; footprint (none) -> Capacitor_SMD:C_0402_1005Metric
- C105: renamed from C?; value 100n -> C; footprint (none) -> Capacitor_SMD:C_0402_1005Metric
- C99: renamed from C?; value 10u -> 0.1uF; footprint (none) -> Capacitor_SMD:C_0402_1005Metric
- L39: renamed from L?; value 1.2u -> 1uH; footprint (none) -> Inductor_SMD:L_0603_1608Metric
- R32: renamed from R?; value 255k -> R; footprint (none) -> Resistor_SMD:R_0603_1608Metric
- R33, R39: renamed from R?; footprint (none) -> Resistor_SMD:R_0603_1608Metric
- R37: renamed from R?; value R -> 5.1k; footprint (none) -> Resistor_SMD:R_0603_1608Metric
- R38, R40: renamed from R?; value 100k -> R; footprint (none) -> Resistor_SMD:R_0603_1608Metric
- U8: renamed from U?; value TPS63020QDSJRQ1 -> BQ25622RYKR; Height 1 -> (none); Manufacturer_Name Texas Instruments -> (none); Manufacturer_Part_Number TPS63020QDSJRQ1 -> (none); Mouser Part Number 595-TPS63020QDSJRQ1 -> (none); Mouser Price/Stock https://www.mouser.co.uk/ProductDetail/Texas-Instruments/TP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 -> (none)
- U9: renamed from U?; value TPS61088RHLR -> ESP32-WROVER-E; Manufacturer_Name Texas Instruments -> (none); Manufacturer_Part_Number TPS61088RHLR -> (none); Mouser Part Number 595-TPS61088RHLR -> (none); Mouser Price/Stock https://www.mouser.co.uk/ProductDetail/Texas-Instruments/TP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 -> (none)
- gave numbers to parts that had none: 43
