File: Hardware/KiCAD/system-testbed/system-testbed.kicad_pcb (KiCad board)
At the start: 2 copper layers, 0 parts

Commit message: Update-Jumper-Schematic
Parts:
- added C1: 1uF, Capacitor_SMD:C_0603_1608Metric, F.Cu at (71.5, 36.1)
- added C10: 47n, Capacitor_SMD:C_0603_1608Metric, F.Cu at (68.6, 97.1)
- added C11: 47n, Capacitor_SMD:C_0603_1608Metric, F.Cu at (72.6, 79.5)
- added C12: 47n, Capacitor_SMD:C_0603_1608Metric, F.Cu at (72.6, 82.1)
- added C13: 47n, Capacitor_SMD:C_0603_1608Metric, F.Cu at (72.6, 84.6)
- added C14: 47n, Capacitor_SMD:C_0603_1608Metric, F.Cu at (72.6, 87.1)
- added C15: 15p, Capacitor_SMD:C_0603_1608Metric, F.Cu at (72.6, 89.6)
- added C16: 10n, Capacitor_SMD:C_0603_1608Metric, F.Cu at (72.6, 92.1)
- added C17: 15p, Capacitor_SMD:C_0603_1608Metric, F.Cu at (72.6, 94.6)
- added C18: 1nF, Capacitor_SMD:C_0603_1608Metric, F.Cu at (72.6, 97.1)
- added C19: 1nF, Capacitor_SMD:C_0603_1608Metric, F.Cu at (76.7, 79.5)
- added C2: 0.1uF, Capacitor_SMD:C_0603_1608Metric, F.Cu at (71.5, 38.7)
- added C20: 1nF, Capacitor_SMD:C_0603_1608Metric, F.Cu at (76.7, 82.1)
- added C21: 1nF, Capacitor_SMD:C_0603_1608Metric, F.Cu at (76.7, 84.6)
- added C22: 220n, Capacitor_SMD:C_0603_1608Metric, F.Cu at (76.7, 87.1)
- added C23: 100pF, Capacitor_SMD:C_0603_1608Metric, F.Cu at (76.7, 89.6)
- added C24: 5.1pF, Capacitor_SMD:C_0603_1608Metric, F.Cu at (68.6, 108.9)
- added C25: 2.2pF, Capacitor_SMD:C_0603_1608Metric, F.Cu at (68.6, 111.5)
- added C26: 5.1pF, Capacitor_SMD:C_0603_1608Metric, F.Cu at (68.6, 114.0)
- added C27: 12pF, Capacitor_SMD:C_0603_1608Metric, F.Cu at (68.6, 116.5)
- added C28: 5.1pF, Capacitor_SMD:C_0603_1608Metric, F.Cu at (68.6, 119.0)
- added C29: 12pF, Capacitor_SMD:C_0603_1608Metric, F.Cu at (68.6, 121.5)
- added C3: 47n, Capacitor_SMD:C_0603_1608Metric, F.Cu at (68.6, 79.5)
- added C30: 100p, Capacitor_SMD:C_0603_1608Metric, F.Cu at (68.6, 124.0)
- added C31: 100p, Capacitor_SMD:C_0603_1608Metric, F.Cu at (68.6, 126.5)
- added C32: 10n, Capacitor_SMD:C_0603_1608Metric, F.Cu at (72.6, 108.9)
- added C33: 10n, Capacitor_SMD:C_0603_1608Metric, F.Cu at (72.6, 111.5)
- added C34: 56p, Capacitor_SMD:C_0603_1608Metric, F.Cu at (72.6, 114.0)
- added C35: 56p, Capacitor_SMD:C_0603_1608Metric, F.Cu at (72.6, 116.5)
- added C36: 39p, Capacitor_SMD:C_0603_1608Metric, F.Cu at (72.6, 119.0)
- added C37: 39p, Capacitor_SMD:C_0603_1608Metric, F.Cu at (72.6, 121.5)
- added C38: 2.2p, Capacitor_SMD:C_0603_1608Metric, F.Cu at (72.6, 124.0)
- added C39: 2.2p, Capacitor_SMD:C_0603_1608Metric, F.Cu at (72.6, 126.5)
- added C4: 47n, Capacitor_SMD:C_0603_1608Metric, F.Cu at (68.6, 82.1)
- added C40: 1nF, Capacitor_SMD:C_0603_1608Metric, F.Cu at (76.7, 108.9)
- added C41: 1nF, Capacitor_SMD:C_0603_1608Metric, F.Cu at (76.7, 111.5)
- added C42: 6.2p, Capacitor_SMD:C_0603_1608Metric, F.Cu at (76.7, 114.0)
- added C43: 6.2p, Capacitor_SMD:C_0603_1608Metric, F.Cu at (76.7, 116.5)
- added C44: 1.2p, Capacitor_SMD:C_0603_1608Metric, F.Cu at (76.7, 119.0)
- added C45: 1.2p, Capacitor_SMD:C_0402_1005Metric, F.Cu at (88.1, 118.0)
- added C46: 1nF, Capacitor_SMD:C_0603_1608Metric, F.Cu at (95.4, 56.0)
- added C47: 10pF, Capacitor_SMD:C_0603_1608Metric, F.Cu at (95.4, 58.5)
- added C48: 33pF, Capacitor_SMD:C_0603_1608Metric, F.Cu at (95.4, 61.0)
- added C49: 1nF, Capacitor_SMD:C_0603_1608Metric, F.Cu at (95.4, 63.5)
- added C5: 47n, Capacitor_SMD:C_0603_1608Metric, F.Cu at (68.6, 84.6)
- added C50: 0.1uF, Capacitor_SMD:C_0603_1608Metric, F.Cu at (95.4, 66.0)
- added C51: 33pF, Capacitor_SMD:C_0603_1608Metric, F.Cu at (99.4, 56.0)
- added C52: 10uF, Capacitor_SMD:C_0603_1608Metric, F.Cu at (99.4, 58.5)
- added C53: 27pF, Capacitor_SMD:C_0603_1608Metric, F.Cu at (99.4, 61.0)
- added C54: 1nF, Capacitor_SMD:C_0603_1608Metric, F.Cu at (99.4, 63.5)
- added C55: 1.8pF, Capacitor_SMD:C_0603_1608Metric, F.Cu at (99.4, 66.0)
- added C56: 27pF, Capacitor_SMD:C_0603_1608Metric, F.Cu at (103.4, 56.0)
- added C57: 1.8pF, Capacitor_SMD:C_0603_1608Metric, F.Cu at (103.4, 58.5)
- added C58: 100pH, Capacitor_SMD:C_0603_1608Metric, F.Cu at (103.4, 61.0)
- added C59: 1nF, Capacitor_SMD:C_0603_1608Metric, F.Cu at (95.4, 36.1)
- added C6: 1.5n, Capacitor_SMD:C_0603_1608Metric, F.Cu at (68.6, 87.1)
- added C60: 10pF, Capacitor_SMD:C_0603_1608Metric, F.Cu at (95.4, 38.7)
- added C61: 33pF, Capacitor_SMD:C_0603_1608Metric, F.Cu at (95.4, 41.2)
- added C62: 1nF, Capacitor_SMD:C_0603_1608Metric, F.Cu at (95.4, 43.7)
- added C63: 0.1uF, Capacitor_SMD:C_0603_1608Metric, F.Cu at (95.4, 46.2)
- added C64: 33pF, Capacitor_SMD:C_0603_1608Metric, F.Cu at (99.4, 36.1)
- added C65: 2.2nH, Capacitor_SMD:C_0603_1608Metric, F.Cu at (99.4, 38.7)
- added C66: 10uF, Capacitor_SMD:C_0603_1608Metric, F.Cu at (99.4, 41.2)
- added C67: 27pF, Capacitor_SMD:C_0603_1608Metric, F.Cu at (99.4, 43.7)
- added C68: 1nF, Capacitor_SMD:C_0603_1608Metric, F.Cu at (99.4, 46.2)
- added C69: 1.8pF, Capacitor_SMD:C_0603_1608Metric, F.Cu at (103.4, 36.1)
- added C7: 47n, Capacitor_SMD:C_0603_1608Metric, F.Cu at (68.6, 89.6)
- added C70: 27pF, Capacitor_SMD:C_0603_1608Metric, F.Cu at (103.4, 38.7)
- added C71: 1.8pF, Capacitor_SMD:C_0603_1608Metric, F.Cu at (103.4, 41.2)
- added C72: 100pH, Capacitor_SMD:C_0603_1608Metric, F.Cu at (103.4, 43.7)
- added C73: 2.2uF, Capacitor_SMD:C_0201_0603Metric, F.Cu at (97.5, 79.2)
- added C74: 1uF, Capacitor_SMD:C_0201_0603Metric, F.Cu at (97.5, 80.9)
- added C75: 10uf, Capacitor_SMD:C_0201_0603Metric, F.Cu at (97.5, 82.7)
- added C76: 4.7uF, Capacitor_SMD:C_0201_0603Metric, F.Cu at (97.5, 84.4)
- added C77: 1uF, Capacitor_SMD:C_0201_0603Metric, F.Cu at (97.5, 86.2)
- added C78: 0.1uF, Capacitor_SMD:C_0201_0603Metric, F.Cu at (97.5, 87.9)
- added C79: 10uF, Capacitor_SMD:C_0201_0603Metric, F.Cu at (97.5, 89.7)
- added C8: 47n, Capacitor_SMD:C_0603_1608Metric, F.Cu at (68.6, 92.1)
- added C80: 47nF, Capacitor_SMD:C_0201_0603Metric, F.Cu at (99.9, 79.2)
- added C81: 20uF, Capacitor_SMD:C_0201_0603Metric, F.Cu at (99.9, 80.9)
- added C9: 47n, Capacitor_SMD:C_0603_1608Metric, F.Cu at (68.6, 94.6)
- added D1: LED, LED_SMD:LED_0201_0603Metric, F.Cu at (107.5, 83.7)
- added D1:1: D, Diode_SMD:D_0603_1608Metric, F.Cu at (24.5, 113.8)
- added D1:2: D, Diode_SMD:D_0603_1608Metric, F.Cu at (24.5, 116.4)
- added D1:3: D, Diode_SMD:D_0603_1608Metric, F.Cu at (24.5, 119.0)
- added D1:4: D, Diode_SMD:D_0603_1608Metric, F.Cu at (24.5, 121.6)
- added D2: LED, LED_SMD:LED_0201_0603Metric, F.Cu at (107.5, 85.5)
- added D2:1: D, Diode_SMD:D_0603_1608Metric, F.Cu at (24.5, 124.2)
- added D2:2: D, Diode_SMD:D_0603_1608Metric, F.Cu at (24.5, 126.7)
- added D2:3: D, Diode_SMD:D_0603_1608Metric, F.Cu at (28.5, 113.8)
- added D2:4: D, Diode_SMD:D_0603_1608Metric, F.Cu at (28.5, 116.4)
- added D3:1: D, Diode_SMD:D_0603_1608Metric, F.Cu at (28.5, 119.0)
- added D3:2: D, Diode_SMD:D_0603_1608Metric, F.Cu at (28.5, 121.6)
- added D3:3: D, Diode_SMD:D_0603_1608Metric, F.Cu at (28.5, 124.2)
- added D3:4: D, Diode_SMD:D_0603_1608Metric, F.Cu at (28.5, 126.7)
- added D4:1: D, Diode_SMD:D_0603_1608Metric, F.Cu at (32.6, 113.8)
- added D4:2: D, Diode_SMD:D_0603_1608Metric, F.Cu at (32.6, 116.4)
- added D4:3: D, Diode_SMD:D_0603_1608Metric, F.Cu at (32.6, 119.0)
- added D4:4: D, Diode_SMD:D_0603_1608Metric, F.Cu at (32.6, 121.6)
- added FL1: LFCN-490, Filter:Filter_Mini-Circuits_FV1206, F.Cu at (89.6, 110.0)
- added FL2: LFCN-160, Filter:Filter_Mini-Circuits_FV1206, F.Cu at (89.6, 114.7)
- added H1: MountingHole_2.2mm_M2_Pad_Via, MountingHole:MountingHole_2.2mm_M2_Pad_Via, F.Cu at (51.9, 115.5)
- added H2: MountingHole_2.2mm_M2_Pad_Via, MountingHole:MountingHole_6.4mm_M6_Pad_Via, F.Cu at (41.8, 119.7)
- added IC1: PCF8575PWR, Package_SO:SSOP-24_5.3x8.2mm_P0.65mm, F.Cu at (36.5, 71.4)
- added J2: Stemma QT, Connector_JST:JST_SH_SM04B-SRSS-TB_1x04-1MP_P1.00mm_Horizontal, F.Cu at (26.9, 56.0)
- added J3: Stemma QT, Connector_JST:JST_SH_SM04B-SRSS-TB_1x04-1MP_P1.00mm_Horizontal, F.Cu at (26.9, 63.7)
- added J4: USB_C_Receptacle_USB2.0_14P, Connector_USB:USB_C_Receptacle_GCT_USB4125-xx-x-0190_6P_TopMnt_Horizontal, F.Cu at (102.2, 95.4)
- added JP1: GAIN_{LOGIC}, Jumper:SolderJumper-3_P1.3mm_Open_RoundedPad1.0x1.5mm_NumberLabels, F.Cu at (80.4, 50.2)
- added JP2: Driver, Jumper:SolderJumper-3_P1.3mm_Bridged12_RoundedPad1.0x1.5mm_NumberLabels, F.Cu at (80.4, 53.8)
- added JP3: GAIN_{R}, Jumper:SolderJumper-3_P1.3mm_Open_RoundedPad1.0x1.5mm_NumberLabels, F.Cu at (80.4, 57.3)
- added JP4: CH_LEFT, Jumper:SolderJumper-2_P1.3mm_Open_RoundedPad1.0x1.5mm, F.Cu at (89.2, 36.7)
- added JP5: CH_MONO_MIX, Jumper:SolderJumper-2_P1.3mm_Bridged_Pad1.0x1.5mm, F.Cu at (89.2, 40.2)
- added JP6: CH_RIGHT, Jumper:SolderJumper-2_P1.3mm_Open_RoundedPad1.0x1.5mm, F.Cu at (89.2, 43.8)
- added JP7: Single V_{CC}, Jumper:SolderJumper-2_P1.3mm_Open_RoundedPad1.0x1.5mm, F.Cu at (100.8, 69.1)
- added JP8: Single V_{CC}, Jumper:SolderJumper-2_P1.3mm_Open_RoundedPad1.0x1.5mm, F.Cu at (100.8, 49.2)
- added L1: 15nH, Inductor_SMD:L_0603_1608Metric, F.Cu at (76.7, 121.5)
- added L10: 220n, Inductor_SMD:L_0603_1608Metric, F.Cu at (80.7, 124.0)
- added L11: 15n, Inductor_SMD:L_0603_1608Metric, F.Cu at (80.7, 126.5)
- added L12: 15n, Inductor_SMD:L_0603_1608Metric, F.Cu at (84.7, 108.9)
- added L13: 43n, Inductor_SMD:L_0603_1608Metric, F.Cu at (84.7, 111.5)
- added L14: 43n, Inductor_SMD:L_0603_1608Metric, F.Cu at (84.7, 114.0)
- added L15: 22n, Inductor_SMD:L_0603_1608Metric, F.Cu at (84.7, 116.5)
- added L16: 22n, Inductor_SMD:L_0603_1608Metric, F.Cu at (84.7, 119.0)
- added L17: 10nH, Inductor_SMD:L_0603_1608Metric, F.Cu at (103.4, 63.5)
- added L18: 20nH, Inductor_SMD:L_0603_1608Metric, F.Cu at (103.4, 66.0)
- added L19: 23nH, Inductor_SMD:L_0603_1608Metric, F.Cu at (107.4, 56.0)
- added L2: 39nH, Inductor_SMD:L_0603_1608Metric, F.Cu at (76.7, 124.0)
- added L20: 2.2nH, Inductor_SMD:L_0603_1608Metric, F.Cu at (107.4, 58.5)
- added L21: 10nH, Inductor_SMD:L_0603_1608Metric, F.Cu at (103.4, 46.2)
- added L22: 20nH, Inductor_SMD:L_0603_1608Metric, F.Cu at (107.4, 36.1)
- added L23: 23nH, Inductor_SMD:L_0603_1608Metric, F.Cu at (107.4, 38.7)
- added L24: 1uH, Inductor_SMD:L_0201_0603Metric, F.Cu at (99.9, 82.7)
- added L3: 27nH, Inductor_SMD:L_0603_1608Metric, F.Cu at (76.7, 126.5)
- added L4: 82nH, Inductor_SMD:L_0603_1608Metric, F.Cu at (80.7, 108.9)
- added L5: 56n, Inductor_SMD:L_0603_1608Metric, F.Cu at (80.7, 111.5)
- added L6: 150n, Inductor_SMD:L_0603_1608Metric, F.Cu at (80.7, 114.0)
- added L7: 27nH, Inductor_SMD:L_0603_1608Metric, F.Cu at (80.7, 116.5)
- added L8: 82nH, Inductor_SMD:L_0603_1608Metric, F.Cu at (80.7, 119.0)
- added L9: 56n, Inductor_SMD:L_0603_1608Metric, F.Cu at (80.7, 121.5)
- added LS1: Speaker, Connector_JST:JST_XH_S2B-XH-A_1x02_P2.50mm_Horizontal, F.Cu at (81.0, 38.2)
- added MK1: ICS-43434, Sensor_Audio:InvenSense_ICS-43434-6_3.5x2.65mm, F.Cu at (85.5, 56.4)
- added P1: SMA, Connector_Coaxial:SMA_Amphenol_901-143_Horizontal, F.Cu at (83.5, 90.8)
- added R1: 47k, Resistor_SMD:R_0603_1608Metric, F.Cu at (71.5, 41.2)
- added R10: 0R, Resistor_SMD:R_0603_1608Metric, F.Cu at (76.7, 92.1)
- added R11: 56k, Resistor_SMD:R_0603_1608Metric, F.Cu at (76.7, 94.6)
- added R12: 18, Resistor_SMD:R_0603_1608Metric, F.Cu at (84.7, 121.5)
- added R13: 18, Resistor_SMD:R_0603_1608Metric, F.Cu at (84.7, 124.0)
- added R14: 1.96k, Resistor_SMD:R_0603_1608Metric, F.Cu at (107.4, 61.0)
- added R15: 6.04k, Resistor_SMD:R_0603_1608Metric, F.Cu at (107.4, 63.5)
- added R16: 0k, Resistor_SMD:R_0603_1608Metric, F.Cu at (107.4, 66.0)
- added R17: 1.96k, Resistor_SMD:R_0603_1608Metric, F.Cu at (107.4, 41.2)
- added R18: 6.04k, Resistor_SMD:R_0603_1608Metric, F.Cu at (107.4, 43.7)
- added R19: 0k, Resistor_SMD:R_0603_1608Metric, F.Cu at (107.4, 46.2)
- added R2: 47k, Resistor_SMD:R_0603_1608Metric, F.Cu at (71.5, 43.7)
- added R20: 0, Resistor_SMD:R_0201_0603Metric, F.Cu at (99.9, 84.4)
- added R21: 1.8M, Resistor_SMD:R_0201_0603Metric, F.Cu at (99.9, 86.2)
- added R22: 10k, Resistor_SMD:R_0201_0603Metric, F.Cu at (99.9, 87.9)
- added R23: 10k, Resistor_SMD:R_0201_0603Metric, F.Cu at (99.9, 89.7)
- added R24: TBD, Resistor_SMD:R_0201_0603Metric, F.Cu at (102.4, 79.2)
- added R25: 10k, Resistor_SMD:R_0201_0603Metric, F.Cu at (102.4, 80.9)
- added R26: 10k, Resistor_SMD:R_0201_0603Metric, F.Cu at (102.4, 82.7)
- added R27: 10k, Resistor_SMD:R_0201_0603Metric, F.Cu at (102.4, 84.4)
- added R28: 10k, Resistor_SMD:R_0201_0603Metric, F.Cu at (102.4, 86.2)
- added R29: 10k, Resistor_SMD:R_0201_0603Metric, F.Cu at (102.4, 87.9)
- added R3: 68, Resistor_SMD:R_0603_1608Metric, F.Cu at (71.5, 46.2)
- added R30: R, Resistor_SMD:R_0201_0603Metric, F.Cu at (102.4, 89.7)
- added R31: R, Resistor_SMD:R_0201_0603Metric, F.Cu at (104.8, 79.2)
- added R32: 5.1k, Resistor_SMD:R_0201_0603Metric, F.Cu at (104.8, 80.9)
- added R33: 5.1k, Resistor_SMD:R_0201_0603Metric, F.Cu at (104.8, 82.7)
- added R4: 100k 5%, Resistor_SMD:R_0603_1608Metric, F.Cu at (71.5, 48.7)
- added R5: 2k, Resistor_SMD:R_0603_1608Metric, F.Cu at (75.5, 36.1)
- added R6: 634k, Resistor_SMD:R_0603_1608Metric, F.Cu at (75.5, 38.7)
- added R7: 330k, Resistor_SMD:R_0603_1608Metric, F.Cu at (75.5, 41.2)
- added R8: 2k, Resistor_SMD:R_0603_1608Metric, F.Cu at (75.5, 43.7)
- added R9: 100k, Resistor_SMD:R_0603_1608Metric, F.Cu at (75.5, 46.2)
- added SW1: RotaryEncoder_Switch, Rotary_Encoder:RotaryEncoder_Bourns_Horizontal_PEC12R-2x17F-Sxxxx, F.Cu at (37.2, 41.1)
- added SW10: 8, Button_Switch_THT:SW_PUSH_6mm_H7.3mm, F.Cu at (35.0, 97.4)
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Routing:
- added copper zone on F.Cu, net +3V3
- added copper zone on B.Cu, net GND
- added copper zone on F.Cu, net GND
Other:
- board outline added: 41 x 25.4 mm
- rule pad_to_mask_clearance: 0.0762 -> 0.05
- board text added: "${REFERENCE}"

Commit message: fix: reannotate schematics for pcb editor use #55
Parts:
- removed C3, C4: 47n, Capacitor_SMD:C_0603_1608Metric
- removed J3: Stemma QT, Connector_JST:JST_SH_SM04B-SRSS-TB_1x04-1MP_P1.00mm_Horizontal
- removed J4: USB_C_Receptacle_USB2.0_14P, Connector_USB:USB_C_Receptacle_GCT_USB4125-xx-x-0190_6P_TopMnt_Horizontal
- removed JP1: GAIN_{LOGIC}, Jumper:SolderJumper-3_P1.3mm_Open_RoundedPad1.0x1.5mm_NumberLabels
- removed SW5: 4, Button_Switch_THT:SW_PUSH_6mm_H7.3mm
- removed SW6: 7, Button_Switch_THT:SW_PUSH_6mm_H7.3mm
- removed U10, U11: GRF5604, Package_DFN_QFN:QFN-16-1EP_3x3mm_P0.5mm_EP1.7x1.7mm_ThermalVias
- removed U12: BQ27427YZFR, capstone-project:DSBGA9-YZF_TEX
- removed U9: SN74LVC2G14DBV, Package_TO_SOT_SMD:SOT-23-6
- added BATT1: M02-JST-2MM-SMT, Connector_PinHeader_2.54mm:PinHeader_1x02_P2.54mm_Vertical, F.Cu at (255.3, -78.1)
- added C100: 10uF, Capacitor_SMD:C_0603_1608Metric, F.Cu at (239.0, -68.6)
- added C101: 47nF, Capacitor_SMD:C_0603_1608Metric, F.Cu at (243.0, -83.7)
- added C102: 20uF, Capacitor_SMD:C_0603_1608Metric, F.Cu at (243.0, -81.2)
- added C82: 33pF, Capacitor_SMD:C_0603_1608Metric, F.Cu at (123.2, 68.5)
- added C83: 1nF, Capacitor_SMD:C_0603_1608Metric, F.Cu at (123.2, 71.0)
- added C84: 0.1uF, Capacitor_SMD:C_0603_1608Metric, F.Cu at (123.2, 73.5)
- added C85: 33pF, Capacitor_SMD:C_0603_1608Metric, F.Cu at (123.2, 76.0)
- added C86: 2.2nH, Capacitor_SMD:C_0603_1608Metric, F.Cu at (123.2, 78.6)
- added C87: 10uF, Capacitor_SMD:C_0603_1608Metric, F.Cu at (127.2, 63.5)
- added C88: 27pF, Capacitor_SMD:C_0603_1608Metric, F.Cu at (127.2, 66.0)
- added C89: 1nF, Capacitor_SMD:C_0603_1608Metric, F.Cu at (127.2, 68.5)
- added C90: 1.8pF, Capacitor_SMD:C_0603_1608Metric, F.Cu at (127.2, 71.0)
- added C91: 27pF, Capacitor_SMD:C_0603_1608Metric, F.Cu at (127.2, 73.5)
- added C92: 1.8pF, Capacitor_SMD:C_0603_1608Metric, F.Cu at (127.2, 76.0)
- added C93: 100pH, Capacitor_SMD:C_0603_1608Metric, F.Cu at (127.2, 78.6)
- added C94: 2.2uF, Capacitor_SMD:C_0603_1608Metric, F.Cu at (239.0, -83.7)
- added C95: 1uF, Capacitor_SMD:C_0603_1608Metric, F.Cu at (239.0, -81.2)
- added C96: 10uf, Capacitor_SMD:C_0603_1608Metric, F.Cu at (239.0, -78.7)
- added C97: 4.7uF, Capacitor_SMD:C_0603_1608Metric, F.Cu at (239.0, -76.2)
- added C98: 1uF, Capacitor_SMD:C_0603_1608Metric, F.Cu at (239.0, -73.6)
- added C99: 0.1uF, Capacitor_SMD:C_0603_1608Metric, F.Cu at (239.0, -71.1)
- added H3: M3, MountingHole:MountingHole_3.2mm_M3_ISO14580_Pad, F.Cu at (41.2, 103.4)
- added H4: M3, MountingHole:MountingHole_3.2mm_M3_ISO14580_Pad, F.Cu at (73.6, 103.4)
- added H5: MountingHole_Pad, MountingHole:MountingHole_3.2mm_M3_ISO14580_Pad, F.Cu at (252.3, -63.8)
- added H6: MountingHole_2.2mm_M2_Pad_Via, MountingHole:MountingHole_2.2mm_M2_Pad_Via, F.Cu at (197.6, -74.1)
- added H7: MountingHole_2.2mm_M2_Pad_Via, MountingHole:MountingHole_6.4mm_M6_Pad_Via, F.Cu at (187.5, -69.9)
- added J1: Stemma QT, Connector_JST:JST_SH_SM04B-SRSS-TB_1x04-1MP_P1.00mm_Horizontal, F.Cu at (223.8, -72.6)
- added J5: USB_C_Receptacle_USB2.0_14P, Connector_USB:USB_C_Receptacle_GCT_USB4125-xx-x-0190_6P_TopMnt_Horizontal, F.Cu at (242.9, -62.5)
- added JP10: SolderJumper_3_Bridged12, Jumper:SolderJumper-2_P1.3mm_Open_RoundedPad1.0x1.5mm, F.Cu at (144.1, -34.1)
- added JP9: Single V_{CC}, Jumper:SolderJumper-2_P1.3mm_Open_RoundedPad1.0x1.5mm, F.Cu at (138.1, 50.4)
- added L25: 100nH, Inductor_SMD:L_0402_1005Metric, F.Cu at (48.5, 94.0)
- added L26: 15nH, Capacitor_SMD:C_0402_1005Metric, F.Cu at (63.5, 80.7)
- added L27: 15nH, Capacitor_SMD:C_0402_1005Metric, F.Cu at (49.1, 85.9)
- added L28: 15nH, Capacitor_SMD:C_0402_1005Metric, F.Cu at (45.0, 95.4)
- added L29: 68nH, Inductor_SMD:L_0402_1005Metric, F.Cu at (59.5, 79.6)
- added L30: 68nH, Inductor_SMD:L_0402_1005Metric, F.Cu at (45.0, 81.8)
- added L31: 68nH, Inductor_SMD:L_0402_1005Metric, F.Cu at (48.9, 96.5)
- added L32: 10nH, Inductor_SMD:L_0402_1005Metric, F.Cu at (123.2, 39.3)
- added L33: 20nH, Inductor_SMD:L_0402_1005Metric, F.Cu at (123.2, 41.8)
- added L34: 23nH, Inductor_SMD:L_0402_1005Metric, F.Cu at (123.2, 44.3)
- added L35: 2.2nH, Inductor_SMD:L_0402_1005Metric, F.Cu at (123.2, 46.8)
- added L36: 10nH, Inductor_SMD:L_0402_1005Metric, F.Cu at (131.2, 63.5)
- added L37: 20nH, Inductor_SMD:L_0402_1005Metric, F.Cu at (131.2, 66.0)
- added L38: 23nH, Inductor_SMD:L_0402_1005Metric, F.Cu at (131.2, 68.5)
- added L39: 1uH, Inductor_SMD:L_0402_1005Metric, F.Cu at (137.6, -35.8)
- added P2: SMA, Connector_Coaxial:SMA_Amphenol_901-144_Vertical, F.Cu at (62.1, 40.6)
- added R34: 0, Resistor_SMD:R_0603_1608Metric, F.Cu at (251.0, -78.7)
- added R35: 5.1k, Resistor_SMD:R_0603_1608Metric, F.Cu at (251.0, -76.2)
- added R36: 5.1k, Resistor_SMD:R_0603_1608Metric, F.Cu at (251.0, -73.6)
- added SW20: DOWN, Button_Switch_THT:SW_PUSH_6mm_H7.3mm, F.Cu at (201.8, -100.7)
- added SW21: LEFT, Button_Switch_THT:SW_PUSH_6mm_H7.3mm, F.Cu at (201.8, -92.1)
- added SW22: RIGHT, Button_Switch_THT:SW_PUSH_6mm_H7.3mm, F.Cu at (201.8, -83.6)
- added SW3: SKY13330-397LF, capstone-project:SKY13330-397LF, F.Cu at (53.3, 48.8)
- added U2: CC1200RHBR, Package_DFN_QFN:QFN-32-1EP_5x5mm_P0.5mm_EP3.45x3.45mm, F.Cu at (61.4, 94.3)
- added U4: TXS0101DBV, Package_TO_SOT_SMD:SOT-23-6, F.Cu at (73.6, 73.5)
- added U5: GRF5604, Package_DFN_QFN:QFN-16-1EP_3x3mm_P0.5mm_EP1.7x1.7mm_ThermalVias, F.Cu at (127.8, 30.6)
- added U6: GRF5604, Package_DFN_QFN:QFN-16-1EP_3x3mm_P0.5mm_EP1.7x1.7mm_ThermalVias, F.Cu at (135.9, 64.9)
- added U7: BQ27427YZFR, capstone-project:DSBGA9-YZF_TEX, F.Cu at (254.7, -71.6)
- added U8: ESP32-WROVER-E, Package_DFN_QFN:QFN-16-1EP_3x3mm_P0.5mm_EP1.7x1.7mm_ThermalVias, F.Cu at (136.3, -26.1)
- added X5: 40 MHz, Crystal:Crystal_SMD_3225-4Pin_3.2x2.5mm, F.Cu at (59.9, 103.1)
- C10, C8: value 47n -> 5.1pF; footprint Capacitor_SMD:C_0603_1608Metric -> Capacitor_SMD:C_0402_1005Metric
- C11, C9: value 47n -> 12pF; footprint Capacitor_SMD:C_0603_1608Metric -> Capacitor_SMD:C_0402_1005Metric
- C12, C13: value 47n -> 100p; footprint Capacitor_SMD:C_0603_1608Metric -> Capacitor_SMD:C_0402_1005Metric
- C14: value 47n -> 10n; footprint Capacitor_SMD:C_0603_1608Metric -> Capacitor_SMD:C_0402_1005Metric
- C15: value 15p -> 10n; footprint Capacitor_SMD:C_0603_1608Metric -> Capacitor_SMD:C_0402_1005Metric
- C16: value 10n -> 56p; footprint Capacitor_SMD:C_0603_1608Metric -> Capacitor_SMD:C_0402_1005Metric
- C17: value 15p -> 56p; footprint Capacitor_SMD:C_0603_1608Metric -> Capacitor_SMD:C_0402_1005Metric
- C18, C19: value 1nF -> 39p; footprint Capacitor_SMD:C_0603_1608Metric -> Capacitor_SMD:C_0402_1005Metric
- C20, C21: value 1nF -> 2.2p; footprint Capacitor_SMD:C_0603_1608Metric -> Capacitor_SMD:C_0402_1005Metric
- C22: value 220n -> 1nF; footprint Capacitor_SMD:C_0603_1608Metric -> Capacitor_SMD:C_0402_1005Metric
- C23: value 100pF -> 1nF; footprint Capacitor_SMD:C_0603_1608Metric -> Capacitor_SMD:C_0402_1005Metric
- C24: value 5.1pF -> 6.2p; footprint Capacitor_SMD:C_0603_1608Metric -> Capacitor_SMD:C_0402_1005Metric
- C25: value 2.2pF -> 6.2p; footprint Capacitor_SMD:C_0603_1608Metric -> Capacitor_SMD:C_0402_1005Metric
- C26: value 5.1pF -> 1.2p; footprint Capacitor_SMD:C_0603_1608Metric -> Capacitor_SMD:C_0402_1005Metric
- C27: value 12pF -> 1.2p; footprint Capacitor_SMD:C_0603_1608Metric -> Capacitor_SMD:C_0402_1005Metric
- C28: value 5.1pF -> 1.5n; footprint Capacitor_SMD:C_0603_1608Metric -> Capacitor_SMD:C_0402_1005Metric
- C29: value 12pF -> 1nF; footprint Capacitor_SMD:C_0603_1608Metric -> Capacitor_SMD:C_0402_1005Metric
- C30, C31: value 100p -> 1nF; footprint Capacitor_SMD:C_0603_1608Metric -> Capacitor_SMD:C_0402_1005Metric
- C32: value 10n -> 1nF; footprint Capacitor_SMD:C_0603_1608Metric -> Capacitor_SMD:C_0402_1005Metric
- C33: value 10n -> 47n; footprint Capacitor_SMD:C_0603_1608Metric -> Capacitor_SMD:C_0402_1005Metric
- C34, C35: value 56p -> 47n; footprint Capacitor_SMD:C_0603_1608Metric -> Capacitor_SMD:C_0402_1005Metric
- C36, C37: value 39p -> 47n; footprint Capacitor_SMD:C_0603_1608Metric -> Capacitor_SMD:C_0402_1005Metric
- C38, C39: value 2.2p -> 100pF; footprint Capacitor_SMD:C_0603_1608Metric -> Capacitor_SMD:C_0402_1005Metric
- C40: value 1nF -> 10n; footprint Capacitor_SMD:C_0603_1608Metric -> Capacitor_SMD:C_0402_1005Metric
- C41, C49: value 1nF -> 47n; footprint Capacitor_SMD:C_0603_1608Metric -> Capacitor_SMD:C_0402_1005Metric
- C42: value 6.2p -> 220n; footprint Capacitor_SMD:C_0603_1608Metric -> Capacitor_SMD:C_0402_1005Metric
- C43: value 6.2p -> 47n; footprint Capacitor_SMD:C_0603_1608Metric -> Capacitor_SMD:C_0402_1005Metric
- C44: value 1.2p -> 1uF; footprint Capacitor_SMD:C_0603_1608Metric -> Capacitor_SMD:C_0402_1005Metric
- C45: value 1.2p -> 47n
- C46: value 1nF -> 15p; footprint Capacitor_SMD:C_0603_1608Metric -> Capacitor_SMD:C_0402_1005Metric
- C47: value 10pF -> 47n; footprint Capacitor_SMD:C_0603_1608Metric -> Capacitor_SMD:C_0402_1005Metric
- C48: value 33pF -> 15p; footprint Capacitor_SMD:C_0603_1608Metric -> Capacitor_SMD:C_0402_1005Metric
- C5: value 47n -> 22pF
- C50: value 0.1uF -> 1uF
- C51: value 33pF -> 47n; footprint Capacitor_SMD:C_0603_1608Metric -> Capacitor_SMD:C_0402_1005Metric
- C52, C66: value 10uF -> 4.7pF; footprint Capacitor_SMD:C_0603_1608Metric -> Capacitor_SMD:C_0402_1005Metric
- C53: value 27pF -> 4.7pF; footprint Capacitor_SMD:C_0603_1608Metric -> Capacitor_SMD:C_0402_1005Metric
- C54: value 1nF -> 4.7pF; footprint Capacitor_SMD:C_0603_1608Metric -> Capacitor_SMD:C_0402_1005Metric
- C55, C57: value 1.8pF -> 18pF; footprint Capacitor_SMD:C_0603_1608Metric -> Capacitor_SMD:C_0402_1005Metric
- C56: value 27pF -> 18pF; footprint Capacitor_SMD:C_0603_1608Metric -> Capacitor_SMD:C_0402_1005Metric
- C58: value 100pH -> 2.7pF; footprint Capacitor_SMD:C_0603_1608Metric -> Capacitor_SMD:C_0402_1005Metric
- C59: value 1nF -> 2.7pF; footprint Capacitor_SMD:C_0603_1608Metric -> Capacitor_SMD:C_0402_1005Metric
- C6: value 1.5n -> 5.1pF; footprint Capacitor_SMD:C_0603_1608Metric -> Capacitor_SMD:C_0402_1005Metric
- C60: value 10pF -> 2.7pF; footprint Capacitor_SMD:C_0603_1608Metric -> Capacitor_SMD:C_0402_1005Metric
- C61: value 33pF -> 18pF; footprint Capacitor_SMD:C_0603_1608Metric -> Capacitor_SMD:C_0402_1005Metric
- C62: value 1nF -> 18pF; footprint Capacitor_SMD:C_0603_1608Metric -> Capacitor_SMD:C_0402_1005Metric
- C63: value 0.1uF -> 18pF; footprint Capacitor_SMD:C_0603_1608Metric -> Capacitor_SMD:C_0402_1005Metric
- C64: value 33pF -> 4.7pF; footprint Capacitor_SMD:C_0603_1608Metric -> Capacitor_SMD:C_0402_1005Metric
- C65: value 2.2nH -> 4.7pF; footprint Capacitor_SMD:C_0603_1608Metric -> Capacitor_SMD:C_0402_1005Metric
- C67, C70: value 27pF -> 1nF
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Connections:
- net /MIC_LRCLK renamed /Audio Subsystem/LR
- C10 pad 1: +3.3V -> /RF Subsystem/LNA_P_{UHF}
- C10 pad 2: GND -> Net-(C10-Pad2)
- C11 pad 1: +3.3V -> /RF Subsystem/LNA_P_{VHF}
- C11 pad 2: GND -> Net-(C11-Pad2)
- C13 pad 1: Net-(U3-DCPL_XOSC) -> +3.3V
- C14 pad 1: Net-(U3-DCPL_PFD_CHP) -> +3.3V
- C15 pad 1: GND -> +3.3V
- C15 pad 2: /RF Subsystem/TRX_X1 -> GND
- C16 pad 1: Net-(U3-DCPL_VCO) -> +3.3V
- C16 pad 2: GND -> Net-(C16-Pad2)
- C17 pad 1: /RF Subsystem/TRX_X2 -> +3.3V
- C17 pad 2: GND -> Net-(C17-Pad2)
- C18 pad 1: /RF Subsystem/RF Frontend/TX_{VHF} -> Net-(C18-Pad1)
- C18 pad 2: Net-(U6-J3) -> /RF Subsystem/PA_{UHF}
- C19 pad 1: /RF Subsystem/RF Frontend/TX_{UHF} -> Net-(C19-Pad1)
- C19 pad 2: Net-(U6-J2) -> /RF Subsystem/PA_{VHF}
- C20 pad 1: /RF Subsystem/RF Frontend/RX_{UHF} -> Net-(C20-Pad1)
- C20 pad 2: Net-(U7-J3) -> Net-(C18-Pad1)
- C21 pad 1: /RF Subsystem/RF Frontend/RX_{VHF} -> Net-(C21-Pad1)
- C21 pad 2: Net-(U7-J2) -> Net-(C19-Pad1)
- C22 pad 1: Net-(U3-DCPL) -> /RF Subsystem/TRX_{SW}
- C22 pad 2: GND -> Net-(C22-Pad2)
- C23 pad 1: Net-(P1-In) -> /RF Subsystem/TRX_{SW}
- C23 pad 2: Net-(U8-J1) -> Net-(C23-Pad2)
- C24 pad 1: /RF Subsystem/RF Frontend/RX_{UHF} -> Net-(C22-Pad2)
- C24 pad 2: Net-(C24-Pad2) -> GND
- C25 pad 1: /RF Subsystem/RF Frontend/RX_{VHF} -> Net-(C23-Pad2)
- C25 pad 2: Net-(C25-Pad2) -> GND
- C26 pad 1: /RF Subsystem/RF Frontend/LNA_N_{UHF} -> Net-(C22-Pad2)
- C26 pad 2: GND -> /RF Subsystem/RF Frontend/UHF 6W PA/RF_{IN}
- C27 pad 1: /RF Subsystem/RF Frontend/LNA_N_{VHF} -> Net-(C23-Pad2)
- C27 pad 2: GND -> /RF Subsystem/RF Frontend/VHF 6W PA/RF_{IN}
- C28 pad 1: /RF Subsystem/RF Frontend/LNA_P_{UHF} -> Net-(U2-LPF1)
- C28 pad 2: Net-(C28-Pad2) -> Net-(U2-LPF0)
- C29 pad 1: /RF Subsystem/RF Frontend/LNA_P_{VHF} -> /RF Subsystem/RF Frontend/RX_{VHF}
- C29 pad 2: Net-(C29-Pad2) -> Net-(SW3-RF2)
- C30 pad 1: +3.3V -> /RF Subsystem/RF Frontend/TX_{VHF}
- C30 pad 2: GND -> Net-(SW3-RF3)
- C31 pad 1: +3.3V -> /RF Subsystem/RF Frontend/RX_{UHF}
- C31 pad 2: GND -> Net-(SW4-RF2)
- C32 pad 1: +3.3V -> /RF Subsystem/RF Frontend/TX_{UHF}
- C32 pad 2: GND -> Net-(SW4-RF3)
- C34 pad 1: +3.3V -> Net-(U2-DCPL_XOSC)
- C34 pad 2: Net-(C34-Pad2) -> GND
- C35 pad 2: Net-(C35-Pad2) -> GND
- C36 pad 1: Net-(C36-Pad1) -> Net-(U2-DCPL_PFD_CHP)
- C36 pad 2: /RF Subsystem/RF Frontend/PA_{UHF} -> GND
- C37 pad 1: Net-(C37-Pad1) -> +3.3V
- C37 pad 2: /RF Subsystem/RF Frontend/PA_{VHF} -> GND
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Routing:
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- removed copper zone on F.Cu, net +3V3
Other:
- board size 41 x 25.4 mm -> 139.6 x 83.4 mm
- rule pad_to_mask_clearance: 0.05 -> 0.0762
- board text added: "BALUN_{RX}"
- board text added: "DIPLEXERS_{RX}"
- board text added: "DIPLEXERS_{TX}"
- board text added: "LNA_{N}"
- board text added: "LNA_{P}"
- board text added: "PA_{EXT}"
- board text added: "RX/TX"
- board text added: "UHF"
- board text added: "VHF"
- board text removed: "${REFERENCE}"

Commit message: fix: allow for DRC use in PCB editor by successful reannotation
Parts:
- removed BATT1: M02-JST-2MM-SMT, Connector_PinHeader_2.54mm:PinHeader_1x02_P2.54mm_Vertical
- removed C100: 10uF, Capacitor_SMD:C_0603_1608Metric
- removed C101: 47nF, Capacitor_SMD:C_0603_1608Metric
- removed C102: 20uF, Capacitor_SMD:C_0603_1608Metric
- removed C97: 4.7uF, Capacitor_SMD:C_0603_1608Metric
- removed C99: 0.1uF, Capacitor_SMD:C_0603_1608Metric
- removed D1, D2: LED, LED_SMD:LED_0201_0603Metric
- removed the H1 at (41.2, 39.3)
- removed the H3 at (41.2, 103.4)
- removed the H4 at (73.6, 103.4)
- removed IC1: PCF8575PWR, Package_SO:SSOP-24_5.3x8.2mm_P0.65mm
- removed J1, J2: Stemma QT, Connector_JST:JST_SH_SM04B-SRSS-TB_1x04-1MP_P1.00mm_Horizontal
- removed J5: USB_C_Receptacle_USB2.0_14P, Connector_USB:USB_C_Receptacle_GCT_USB4125-xx-x-0190_6P_TopMnt_Horizontal
- removed JP10: SolderJumper_3_Bridged12, Jumper:SolderJumper-2_P1.3mm_Open_RoundedPad1.0x1.5mm
- removed L39: 1uH, Inductor_SMD:L_0402_1005Metric
- removed R20, R25, R28, R34: 0, Resistor_SMD:R_0603_1608Metric
- removed R21: 1.8M, Resistor_SMD:R_0603_1608Metric
- removed R22, R23, R26, R27, R29, R30, R31: 10k, Resistor_SMD:R_0603_1608Metric
- removed R24: TBD, Resistor_SMD:R_0603_1608Metric
- removed R35, R36: 5.1k, Resistor_SMD:R_0603_1608Metric
- removed SW1: RotaryEncoder_Switch, Rotary_Encoder:RotaryEncoder_Bourns_Horizontal_PEC12R-2x17F-Sxxxx
- removed SW10: *, Button_Switch_THT:SW_PUSH_6mm_H7.3mm
- removed SW11: 2, Button_Switch_THT:SW_PUSH_6mm_H7.3mm
- removed SW12: 5, Button_Switch_THT:SW_PUSH_6mm_H7.3mm
- removed SW13: 8, Button_Switch_THT:SW_PUSH_6mm_H7.3mm
- removed SW14: 0, Button_Switch_THT:SW_PUSH_6mm_H7.3mm
- removed SW15: 3, Button_Switch_THT:SW_PUSH_6mm_H7.3mm
- removed SW16: 6, Button_Switch_THT:SW_PUSH_6mm_H7.3mm
- removed SW17: 9, Button_Switch_THT:SW_PUSH_6mm_H7.3mm
- removed SW18: #, Button_Switch_THT:SW_PUSH_6mm_H7.3mm
- removed SW19: UP, Button_Switch_THT:SW_PUSH_6mm_H7.3mm
- removed SW20: DOWN, Button_Switch_THT:SW_PUSH_6mm_H7.3mm
- removed SW21: LEFT, Button_Switch_THT:SW_PUSH_6mm_H7.3mm
- removed SW22: RIGHT, Button_Switch_THT:SW_PUSH_6mm_H7.3mm
- removed SW7: 1, Button_Switch_THT:SW_PUSH_6mm_H7.3mm
- removed SW8: 4, Button_Switch_THT:SW_PUSH_6mm_H7.3mm
- removed SW9: 7, Button_Switch_THT:SW_PUSH_6mm_H7.3mm
- removed U7: BQ27427YZFR, capstone-project:DSBGA9-YZF_TEX
- removed U9(Note-checkpinsinsymboleditor)1: BQ25622RYKR, capstone-project:WQFN-HR18__RYK_TEX
- removed VR1: RK09711110EL, capstone-project:RK09711110EL
- removed X2, X3, X4: EYESPI, capstone-project:Adafruit EYESPI FPC Connector
- added BATT301: M02-JST-2MM-SMT, Connector_JST:JST_GH_BM02B-GHS-TBT_1x02-1MP_P1.25mm_Vertical, F.Cu at (92.0, 163.7)
- added C106: 0.1u, Capacitor_SMD:C_0603_1608Metric, F.Cu at (69.2, 78.9)
- added C394: 2.2uF, Capacitor_SMD:C_0603_1608Metric, F.Cu at (80.4, 151.9)
- added C395: 1uF, Capacitor_SMD:C_0603_1608Metric, F.Cu at (77.2, 155.1)
- added C400: 10uf, Capacitor_SMD:C_0603_1608Metric, F.Cu at (87.1, 155.1)
- added C401: 4.7uF, Capacitor_SMD:C_0603_1608Metric, F.Cu at (84.2, 148.9)
- added C403: 47nF, Capacitor_SMD:C_0603_1608Metric, F.Cu at (91.3, 148.1)
- added C404: 0.1uF, Capacitor_SMD:C_0603_1608Metric, F.Cu at (89.8, 145.6)
- added C405: 10uF, Capacitor_SMD:C_0603_1608Metric, F.Cu at (88.2, 145.6)
- added C406: 1uF, Capacitor_SMD:C_0603_1608Metric, F.Cu at (85.9, 146.3)
- added C407: 20uF, Capacitor_SMD:C_0603_1608Metric, F.Cu at (91.1, 154.1)
- added C409: C, Capacitor_SMD:C_0603_1608Metric, F.Cu at (131.9, 142.2)
- added C410: C, Capacitor_SMD:C_0603_1608Metric, F.Cu at (131.9, 144.7)
- added C411: C, Capacitor_SMD:C_0603_1608Metric, F.Cu at (131.9, 147.3)
- added C445: 1uF, Capacitor_SMD:C_0603_1608Metric, F.Cu at (89.4, 154.1)
- added D302: ESDA25P35-1U1M, capstone-project:TVS_ESDA25P35-1U1M, F.Cu at (126.2, 132.4)
- added D303: LED, LED_SMD:LED_0603_1608Metric, F.Cu at (97.9, 155.2)
- added D304: LED, LED_SMD:LED_0603_1608Metric, F.Cu at (81.1, 147.6)
- added D305: ESDA25P35-1U1M, capstone-project:TVS_ESDA25P35-1U1M, F.Cu at (126.2, 135.0)
- added D306: ESDA25P35-1U1M, capstone-project:TVS_ESDA25P35-1U1M, F.Cu at (126.2, 137.6)
- added H1: M3, MountingHole:MountingHole_3.2mm_M3_ISO14580_Pad, F.Cu at (67.7, 130.5)
- added H1: MountHole, MountingHole:MountingHole_3.2mm_M3_ISO14580_Pad, F.Cu at (50.2, 54.4)
- added H10: M3, MountingHole:MountingHole_3.2mm_M3_ISO14580_Pad, F.Cu at (175.5, 45.2)
- added H11: M3, MountingHole:MountingHole_3.2mm_M3_ISO14580_Pad, F.Cu at (144.1, 92.9)
- added H12: M3, MountingHole:MountingHole_3.2mm_M3_ISO14580_Pad, F.Cu at (175.9, 92.9)
- added H13: M3, MountingHole:MountingHole_3.2mm_M3_ISO14580_Pad, F.Cu at (193.1, 131.3)
- added H14: M3, MountingHole:MountingHole_3.2mm_M3_ISO14580_Pad, F.Cu at (225.0, 131.2)
- added H15: M3, MountingHole:MountingHole_3.2mm_M3_ISO14580_Pad, F.Cu at (193.0, 147.3)
- added H16: M3, MountingHole:MountingHole_3.2mm_M3_ISO14580_Pad, F.Cu at (225.0, 147.6)
- added H2: M3, MountingHole:MountingHole_3.2mm_M3_ISO14580_Pad, F.Cu at (82.5, 54.4)
- added H3: M3, MountingHole:MountingHole_3.2mm_M3_ISO14580_Pad, F.Cu at (99.4, 130.4)
- added H3: MountHole, MountingHole:MountingHole_3.2mm_M3_ISO14580_Pad, F.Cu at (50.2, 86.5)
- added H305: MountHole, MountingHole:MountingHole_3.2mm_M3_ISO14580_Pad, F.Cu at (48.0, 130.5)
- added H306: MountHole, MountingHole:MountingHole_3.2mm_M3_ISO14580_Pad, F.Cu at (31.8, 130.6)
- added H307: MountHole, MountingHole:MountingHole_3.2mm_M3_ISO14580_Pad, F.Cu at (32.0, 162.9)
- added H308: MountHole, MountingHole:MountingHole_3.2mm_M3_ISO14580_Pad, F.Cu at (47.8, 162.9)
- added H4: M3, MountingHole:MountingHole_3.2mm_M3_ISO14580_Pad, F.Cu at (67.7, 162.4)
- added H4: MountHole, MountingHole:MountingHole_3.2mm_M3_ISO14580_Pad, F.Cu at (82.5, 86.5)
- added H8: M3, MountingHole:MountingHole_3.2mm_M3_ISO14580_Pad, F.Cu at (99.8, 162.4)
- added H9: M3, MountingHole:MountingHole_3.2mm_M3_ISO14580_Pad, F.Cu at (143.8, 45.2)
- added IC2: PCF8575PWR, Package_SO:SSOP-24_5.3x8.2mm_P0.65mm, F.Cu at (154.4, 65.4)
- added J305: 217177-0001, capstone-project:2171770001, F.Cu at (67.1, 149.9)
- added J4: Conn_01x08_Pin, Connector_JST:JST_EH_B8B-EH-A_1x08_P2.50mm_Vertical, F.Cu at (199.8, 149.2)
- added J7: Stemma QT, Connector_JST:JST_SH_SM04B-SRSS-TB_1x04-1MP_P1.00mm_Horizontal, F.Cu at (75.7, 87.4)
- added J9: Display Pin Socket, Connector_PinHeader_2.54mm:PinHeader_1x11_P2.54mm_Vertical, F.Cu at (175.5, 49.4)
- added L339: 1uH, Inductor_SMD:L_0603_1608Metric, F.Cu at (92.5, 151.1)
- added LED301: LTST-C190KRKT, capstone-project:LTST-C190KRKT, F.Cu at (133.3, 162.0)
- added Q302: 2N7002, Package_TO_SOT_SMD:SOT-23, F.Cu at (128.3, 170.8)
- added R321: 1.8M, Resistor_SMD:R_0603_1608Metric, F.Cu at (138.7, 133.9)
- added R322: bias, Resistor_SMD:R_0603_1608Metric, F.Cu at (135.1, 167.7)
- added R323: 10k, Resistor_SMD:R_0603_1608Metric, F.Cu at (138.7, 138.9)
- added R324: 10k, Resistor_SMD:R_0603_1608Metric, F.Cu at (111.9, 170.1)
- added R325: 10k, Resistor_SMD:R_0603_1608Metric, F.Cu at (122.3, 127.6)
- added R330: 0, Resistor_SMD:R_0603_1608Metric, F.Cu at (112.8, 160.0)
- added R334: 1, Resistor_SMD:R_0603_1608Metric, F.Cu at (112.8, 162.5)
- added R335: TBD, Resistor_SMD:R_0603_1608Metric, F.Cu at (84.2, 152.1)
- added R337: 10k, Resistor_SMD:R_0603_1608Metric, F.Cu at (121.0, 157.6)
- added R339: 10k, Resistor_SMD:R_0603_1608Metric, F.Cu at (123.5, 157.6)
- added R342: 10k, Resistor_SMD:R_0603_1608Metric, F.Cu at (100.5, 155.9)
- added R343: 10k, Resistor_SMD:R_0603_1608Metric, F.Cu at (77.2, 147.6)
- added R344: 10k, Resistor_SMD:R_0603_1608Metric, F.Cu at (95.3, 153.1)
- added R345: R, Resistor_SMD:R_0603_1608Metric, F.Cu at (88.1, 157.8)
- added R346: R, Resistor_SMD:R_0603_1608Metric, F.Cu at (91.9, 157.8)
- added R347: 0, Resistor_SMD:R_0603_1608Metric, F.Cu at (111.5, 165.8)
- added R348: 0, Resistor_SMD:R_0603_1608Metric, F.Cu at (96.1, 150.3)
- added R351: R, Resistor_SMD:R_0603_1608Metric, F.Cu at (131.9, 149.8)
- added R352: R, Resistor_SMD:R_0603_1608Metric, F.Cu at (131.9, 152.3)
- added R353: R, Resistor_SMD:R_0603_1608Metric, F.Cu at (131.9, 154.8)
- added S301: 100SP1T1B4M2QE, capstone-project:SW_100SP1T1B4M2QE, F.Cu at (79.4, 162.4)
- added SW28: SW_Push, Button_Switch_SMD:SW_SPST_EVQP2_MiddlePushTravel_H2.5mm, F.Cu at (74.7, 78.9)
- added SW30: #, Button_Switch_SMD:SW_Push_1P1T_NO_CK_KMR2, F.Cu at (143.6, 88.0)
- added SW31: 1, Button_Switch_SMD:SW_Push_1P1T_NO_CK_KMR2, F.Cu at (143.6, 77.0)
- added SW32: 4, Button_Switch_SMD:SW_Push_1P1T_NO_CK_KMR2, F.Cu at (143.6, 80.7)
- added SW33: 7, Button_Switch_SMD:SW_Push_1P1T_NO_CK_KMR2, F.Cu at (143.6, 84.3)
- added SW34: 0, Button_Switch_SMD:SW_Push_1P1T_NO_CK_KMR2, F.Cu at (149.2, 88.0)
- added SW35: 2, Button_Switch_SMD:SW_Push_1P1T_NO_CK_KMR2, F.Cu at (149.2, 77.0)
- added SW36: 5, Button_Switch_SMD:SW_Push_1P1T_NO_CK_KMR2, F.Cu at (149.2, 80.7)
- added SW37: 8, Button_Switch_SMD:SW_Push_1P1T_NO_CK_KMR2, F.Cu at (149.2, 84.4)
- added SW38: *, Button_Switch_SMD:SW_Push_1P1T_NO_CK_KMR2, F.Cu at (154.9, 88.0)
- added SW39: 3, Button_Switch_SMD:SW_Push_1P1T_NO_CK_KMR2, F.Cu at (154.9, 77.0)
- added SW40: 6, Button_Switch_SMD:SW_Push_1P1T_NO_CK_KMR2, F.Cu at (154.9, 80.7)
- added SW41: 9, Button_Switch_SMD:SW_Push_1P1T_NO_CK_KMR2, F.Cu at (154.9, 84.4)
- added SW42: RIGHT, Button_Switch_SMD:SW_Push_1P1T_NO_CK_KMR2, F.Cu at (201.7, 95.7)
- added SW43: UP, Button_Switch_SMD:SW_Push_1P1T_NO_CK_KMR2, F.Cu at (195.6, 93.0)
- added SW44: DOWN, Button_Switch_SMD:SW_Push_1P1T_NO_CK_KMR2, F.Cu at (195.6, 98.6)
- added SW45: LEFT, Button_Switch_SMD:SW_Push_1P1T_NO_CK_KMR2, F.Cu at (189.5, 95.7)
- added SW5: SW_Push, Button_Switch_SMD:SW_SPST_EVQP2_MiddlePushTravel_H2.5mm, F.Cu at (57.8, 78.9)
- added TH301: Thermistor_NTC, Resistor_THT:R_Axial_DIN0204_L3.6mm_D1.6mm_P2.54mm_Vertical, F.Cu at (94.9, 158.0)
- added TP1: +3.3V, TestPoint:TestPoint_Pad_D1.0mm, B.Cu at (262.7, 88.0)
- added TP10: X1, TestPoint:TestPoint_Pad_D1.0mm, F.Cu at (248.8, 96.7)
- added TP11: X2, TestPoint:TestPoint_Pad_D1.0mm, F.Cu at (258.0, 97.1)
- added TP12: TRX_SW, TestPoint:TestPoint_Pad_D1.0mm, F.Cu at (263.9, 66.4)
- added TP13: TRX_SW_{+2.5V}, TestPoint:TestPoint_Pad_D1.0mm, F.Cu at (266.6, 53.4)
- added TP14: PA SHUTDOWN, TestPoint:TestPoint_Pad_D1.0mm, F.Cu at (254.7, 55.9)
- added TP15: LNA_P_{2m}, TestPoint:TestPoint_Pad_D1.0mm, F.Cu at (239.3, 83.8)
- added TP16: LNA_P_{70cm}, TestPoint:TestPoint_Pad_D1.0mm, F.Cu at (239.3, 72.6)
- added TP17: LNA_N_{2m}, TestPoint:TestPoint_Pad_D1.0mm, F.Cu at (239.5, 92.2)
- added TP18: LNA_N_{70cm}, TestPoint:TestPoint_Pad_D1.0mm, F.Cu at (239.3, 81.3)
- added TP19: PA_{2m}, TestPoint:TestPoint_Pad_D1.0mm, F.Cu at (254.3, 74.5)
- added TP2: NRST, TestPoint:TestPoint_Pad_D1.0mm, B.Cu at (266.8, 88.0)
- added TP20: PA_{70cm}, TestPoint:TestPoint_Pad_D1.0mm, F.Cu at (256.6, 74.5)
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Connections:
- net /TRX_GPIO0 renamed /RF Subsystem/TRX_GPIO0
- net /TRX_GPIO2 renamed /RF Subsystem/TRX_GPIO2
- net /TRX_MISO renamed /RF Subsystem/TRX_MISO
- net /TRX_MOSI renamed /RF Subsystem/TRX_MOSI
- net /TRX_NCS renamed /RF Subsystem/TRX_NCS
- net /TRX_NRST renamed /RF Subsystem/TRX_NRST
- net /TRX_SCLK renamed /RF Subsystem/TRX_SCLK
- C1 pad 1: +3.3V -> GND
- C1 pad 2: GND -> Net-(U8-EN)
- C2 pad 1: +3.3V -> GND
- C2 pad 2: GND -> +3.3V
- C5 pad 1: /BCLK -> Net-(C5-Pad1)
- C71 pad 1: +5V -> +3.3V
- C84 pad 1: +5V -> +3.3V
- C94 pad 1: Net-(U7-VDD) -> GND
- C94 pad 2: GND -> Net-(U8-EN)
- C95 pad 1: /Power Subsystem/Battery(+) -> GND
- C95 pad 2: GND -> +3.3V
- C96 pad 1: /Power Subsystem/Batt (+) -> GND
- C96 pad 2: GND -> +3.3V
- C98 pad 1: GND -> Net-(C98-Pad1)
- C98 pad 2: Net-(U9(Note-checkpinsinsymboleditor)1-VBUS) -> GND
- H6 pad 1: (no net) -> GND
- H7 pad 1: (no net) -> GND
- JP8 pad 1: +5V -> +3.3V
- JP9 pad 1: +5V -> +3.3V
- L33 pad 1: +5V -> +3.3V
- L37 pad 1: +5V -> +3.3V
- R1 pad 1: /Audio Subsystem/LR -> Net-(R1-Pad1)
- R1 pad 2: GND -> Net-(U8-EN)
- R2 pad 1: Net-(MK1-SD) -> Net-(U8-EN)
- R2 pad 2: GND -> +3.3V
- R3 pad 1: Net-(MK1-SD) -> Net-(C5-Pad1)
- R3 pad 2: /MIC_DOUT -> +3.3V
- R32 pad 1: /Power Subsystem/TS_BIAS -> Net-(R32-Pad1)
- R32 pad 2: /Power Subsystem/TS -> Net-(U8-EN)
- R33 pad 1: /Power Subsystem/TS -> Net-(U8-EN)
- R33 pad 2: GND -> +3.3V
- R4 pad 1: Net-(JP3-C) -> +3.3V
- R4 pad 2: /Audio Subsystem/~{SD_MODE} -> Net-(C98-Pad1)
- R5 pad 1: Net-(JP2-C) -> /Human-Machine Interface/ENC_CLK
- R5 pad 2: Net-(JP4-B) -> Net-(C98-Pad1)
- R6 pad 1: Net-(JP6-A) -> /Human-Machine Interface/ENC_DT
- R6 pad 2: /~{AMP_SD} -> Net-(C5-Pad1)
- U8 pad 1: unconnected-(U8-GND-Pad1) -> GND
- U8 pad 11: unconnected-(U8-26_HSPI_DC-Pad11) -> /MCU/HSPI_DC
- U8 pad 13: unconnected-(U8-14_HSPI_SCLK-Pad13) -> /MCU/HSPI_SCLK
- U8 pad 15: unconnected-(U8-GND-Pad15) -> GND
- U8 pad 16: unconnected-(U8-13_HSPI_MOSI-Pad16) -> /MCU/HSPI_MOSI
- U8 pad 2: unconnected-(U8-3V3-Pad2) -> +3.3V
- U8 pad 3: unconnected-(U8-EN-Pad3) -> Net-(U8-EN)
- U8 pad 5: unconnected-(U8-39_X_INT-Pad5) -> /MCU/XTND_INT
- U8 pad 6: unconnected-(U8-34_VSPI_GDO0-Pad6) -> /MCU/VSPI_GDO0
- U8 pad 7: unconnected-(U8-35_VSPI_GDO2-Pad7) -> /MCU/VSPI_GDO2
- U8 pad 8: unconnected-(U8-32_VSPI_CS-Pad8) -> /MCU/VSPI_CS
Routing:
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Other:
- board size 139.6 x 83.4 mm -> 244.7 x 127.4 mm
- board text added: "Audio Modulino"
- board text added: "BMS"
- board text added: "ESP32 Modulino"
- board text added: "HMI Modulino"
- board text added: "Plug&Make"
- board text added: "Power Modulinos"
- board text added: "RF Modulino"
- board text added: "USB-PD"
- board text added: "Z MATCHING"
