File: Hardware/KiCAD/system-testbed/system-testbed.kicad_pcb (KiCad board)
At the start: 2 copper layers, 244.7 x 127.4 mm, 330 parts, among them IC2 PCF8575PWR, J305 217177-0001, J4 Conn_01x08_Pin, J7 Stemma QT, J9 Display Pin Socket, P1 SMA, P2 SMA, Q302 2N7002, SW28 SW_Push, SW3 SKY13330-397LF, SW30 #, SW31 1, SW32 4, SW33 7, SW34 0, SW35 2, SW36 5, SW37 8, SW38 *, SW39 3, SW4 SKY13330-397LF, SW40 6, SW41 9, SW42 RIGHT, SW43 UP, SW44 DOWN, SW45 LEFT, SW5 SW_Push, U1 PEC11J-9215F-S0015, U2 CC1200RHBR, U3 LP5907MFX-2.5, U307 STUSB4500QTR, U308 BQ27427YZFR, U309 BQ25622RYKR, U312 TPS63020QDSJRQ1, U4 TXS0101DBV, U5 GRF5604, U6 GRF5604, U8 ESP32-WROVER-E, X1 EYESPI, X11 EYESPI, X12 EYESPI, X309 EYESPI, X5 40 MHz, X6 EYESPI, X7 EYESPI, X8 EYESPI, X9 EYESPI

Commit message: feat: separate RF subsystems for testing using SMA edge launches in testbed KiCAD project #65 #34 #45
Parts:
- removed BATT301: M02-JST-2MM-SMT, Connector_JST:JST_GH_BM02B-GHS-TBT_1x02-1MP_P1.25mm_Vertical
- removed C1, C106, C94, C96: 0.1u, Capacitor_SMD:C_0603_1608Metric
- removed C2, C95: 10u, Capacitor_SMD:C_0603_1608Metric
- removed C39: 100pF, Capacitor_SMD:C_0402_1005Metric
- removed C394: 2.2uF, Capacitor_SMD:C_0603_1608Metric
- removed C395, C406, C445: 1uF, Capacitor_SMD:C_0603_1608Metric
- removed C400: 10uf, Capacitor_SMD:C_0603_1608Metric
- removed C401: 4.7uF, Capacitor_SMD:C_0603_1608Metric
- removed C403: 47nF, Capacitor_SMD:C_0603_1608Metric
- removed C404: 0.1uF, Capacitor_SMD:C_0603_1608Metric
- removed C405: 10uF, Capacitor_SMD:C_0603_1608Metric
- removed C407: 20uF, Capacitor_SMD:C_0603_1608Metric
- removed C409, C410, C411: C, Capacitor_SMD:C_0603_1608Metric
- removed C5, C98: 0.01uF, Capacitor_SMD:C_0603_1608Metric
- removed D1:1, D1:2, D1:3, D1:4, D2:1, D2:2, D2:3, D2:4, D3:1, D3:2, D3:3, D3:4, D4:1, D4:2, D4:3, D4:4: D, Diode_SMD:D_0603_1608Metric
- removed D302, D305, D306: ESDA25P35-1U1M, capstone-project:TVS_ESDA25P35-1U1M
- removed D303, D304: LED, LED_SMD:LED_0603_1608Metric
- removed the H1 at (67.7, 130.5)
- removed the H1 at (50.2, 54.4)
- removed H10, H11, H12, H13, H14, H15, H16, H7, H9: M3, MountingHole:MountingHole_3.2mm_M3_ISO14580_Pad
- removed the H2 at (82.5, 54.4)
- removed the H3 at (99.4, 130.4)
- removed the H3 at (50.2, 86.5)
- removed H305, H306, H307, H308: MountHole, MountingHole:MountingHole_3.2mm_M3_ISO14580_Pad
- removed the H4 at (67.7, 162.4)
- removed the H4 at (82.5, 86.5)
- removed IC2: PCF8575PWR, Package_SO:SSOP-24_5.3x8.2mm_P0.65mm
- removed J305: 217177-0001, capstone-project:2171770001
- removed J7: Stemma QT, Connector_JST:JST_SH_SM04B-SRSS-TB_1x04-1MP_P1.00mm_Horizontal
- removed J9: Display Pin Socket, Connector_PinHeader_2.54mm:PinHeader_1x11_P2.54mm_Vertical
- removed JP2: GAIN_{LOGIC}, Jumper:SolderJumper-3_P1.3mm_Open_RoundedPad1.0x1.5mm_NumberLabels
- removed JP4: GAIN_{R}, Jumper:SolderJumper-3_P1.3mm_Open_RoundedPad1.0x1.5mm_NumberLabels
- removed JP5: CH_LEFT, Jumper:SolderJumper-2_P1.3mm_Open_RoundedPad1.0x1.5mm
- removed JP6: CH_MONO_MIX, Jumper:SolderJumper-2_P1.3mm_Bridged_Pad1.0x1.5mm
- removed JP7: CH_RIGHT, Jumper:SolderJumper-2_P1.3mm_Open_RoundedPad1.0x1.5mm
- removed L339: 1uH, Inductor_SMD:L_0603_1608Metric
- removed LED301: LTST-C190KRKT, capstone-project:LTST-C190KRKT
- removed LS1: Speaker, Connector_JST:JST_EH_B2B-EH-A_1x02_P2.50mm_Vertical
- removed MK1: ICS-43434, Sensor_Audio:InvenSense_ICS-43434-6_3.5x2.65mm
- removed P2: SMA, Connector_Coaxial:SMA_Amphenol_901-144_Vertical
- removed Q302: 2N7002, Package_TO_SOT_SMD:SOT-23
- removed R1, R2, R3, R32, R323, R324, R325, R33, R337, R339, R342, R343, R344, R4, R5, R6: 10k, Resistor_SMD:R_0603_1608Metric
- removed R321: 1.8M, Resistor_SMD:R_0603_1608Metric
- removed R322: bias, Resistor_SMD:R_0603_1608Metric
- removed R330, R347, R348: 0, Resistor_SMD:R_0603_1608Metric
- removed R334: 1, Resistor_SMD:R_0603_1608Metric
- removed R335: TBD, Resistor_SMD:R_0603_1608Metric
- removed R345, R346, R351, R352, R353: R, Resistor_SMD:R_0603_1608Metric
- removed R8: 2k, Resistor_SMD:R_0603_1608Metric
- removed R9: 100k, Resistor_SMD:R_0603_1608Metric
- removed S301: 100SP1T1B4M2QE, capstone-project:SW_100SP1T1B4M2QE
- removed SW28: SW_Push, Button_Switch_SMD:SW_SPST_EVQP2_MiddlePushTravel_H2.5mm
- removed SW30: #, Button_Switch_SMD:SW_Push_1P1T_NO_CK_KMR2
- removed SW31: 1, Button_Switch_SMD:SW_Push_1P1T_NO_CK_KMR2
- removed SW32: 4, Button_Switch_SMD:SW_Push_1P1T_NO_CK_KMR2
- removed SW33: 7, Button_Switch_SMD:SW_Push_1P1T_NO_CK_KMR2
- removed SW34: 0, Button_Switch_SMD:SW_Push_1P1T_NO_CK_KMR2
- removed SW35: 2, Button_Switch_SMD:SW_Push_1P1T_NO_CK_KMR2
- removed SW36: 5, Button_Switch_SMD:SW_Push_1P1T_NO_CK_KMR2
- removed SW37: 8, Button_Switch_SMD:SW_Push_1P1T_NO_CK_KMR2
- removed SW38: *, Button_Switch_SMD:SW_Push_1P1T_NO_CK_KMR2
- removed SW39: 3, Button_Switch_SMD:SW_Push_1P1T_NO_CK_KMR2
- removed SW40: 6, Button_Switch_SMD:SW_Push_1P1T_NO_CK_KMR2
- removed SW41: 9, Button_Switch_SMD:SW_Push_1P1T_NO_CK_KMR2
- removed SW42: RIGHT, Button_Switch_SMD:SW_Push_1P1T_NO_CK_KMR2
- removed SW43: UP, Button_Switch_SMD:SW_Push_1P1T_NO_CK_KMR2
- removed SW44: DOWN, Button_Switch_SMD:SW_Push_1P1T_NO_CK_KMR2
- removed SW45: LEFT, Button_Switch_SMD:SW_Push_1P1T_NO_CK_KMR2
- removed TH301: Thermistor_NTC, Resistor_THT:R_Axial_DIN0204_L3.6mm_D1.6mm_P2.54mm_Vertical
- removed TP14: PA SHUTDOWN, TestPoint:TestPoint_Pad_D1.0mm
- removed TP15: LNA_P_{2m}, TestPoint:TestPoint_Pad_D1.0mm
- removed TP16: LNA_P_{70cm}, TestPoint:TestPoint_Pad_D1.0mm
- removed TP17: LNA_N_{2m}, TestPoint:TestPoint_Pad_D1.0mm
- removed TP18: LNA_N_{70cm}, TestPoint:TestPoint_Pad_D1.0mm
- removed TP19: PA_{2m}, TestPoint:TestPoint_Pad_D1.0mm
- removed TP20: PA_{70cm}, TestPoint:TestPoint_Pad_D1.0mm
- removed TP329, TP330, TP331, TP332, TP333, TP334, TP335, TP336, TP337, TP338: TestPoint, TestPoint:TestPoint_Loop_D2.60mm_Drill1.6mm_Beaded
- removed U1: PEC11J-9215F-S0015, capstone-project:PEC11J9215FS0015
- removed U307: STUSB4500QTR, capstone-project:STUSB4500QTR
- removed U308: BQ27427YZFR, capstone-project:DSBGA9-YZF_TEX
- removed U309: BQ25622RYKR, capstone-project:WQFN-HR18__RYK_TEX
- removed U312: TPS63020QDSJRQ1, capstone-project:TPS63020DSJR
- removed U8: ESP32-WROVER-E, capstone-project:ESP32-WROVER-IE
- removed X11, X12, X309, X6, X7, X8, X9: EYESPI, capstone-project:Adafruit EYESPI FPC Connector
- added C81: 1nF, Capacitor_SMD:C_0402_1005Metric, F.Cu at (189.7, 58.2)
- added G***: LOGO, capstone-project:LOGO, F.Cu at (188.1, 74.8)
- added G***: LOGO, capstone-project:LOGO, F.Cu at (63.5, 73.6)
- added G***: LOGO, capstone-project:LOGO, F.Cu at (133.0, 73.9)
- added H1: M3, MountingHole:MountingHole_3.2mm_M3_ISO14580_Pad, F.Cu at (108.6, 49.6)
- added H1: M3, MountingHole:MountingHole_3.2mm_M3_ISO14580_Pad, F.Cu at (69.8, 49.2)
- added H3: M3, MountingHole:MountingHole_3.2mm_M3_ISO14580_Pad, F.Cu at (69.8, 81.3)
- added H3: M3, MountingHole:MountingHole_3.2mm_M3_ISO14580_Pad, F.Cu at (140.6, 49.6)
- added H4: M3, MountingHole:MountingHole_3.2mm_M3_ISO14580_Pad, F.Cu at (108.7, 81.5)
- added H5: M3, MountingHole:MountingHole_3.2mm_M3_ISO14580_Pad, F.Cu at (179.1, 49.6)
- added J2: Conn_01x06_Pin, Connector_PinHeader_2.54mm:PinHeader_1x06_P2.54mm_Vertical, B.Cu at (131.3, 46.6)
- added J3: Conn_01x06_Pin, Connector_PinHeader_2.54mm:PinHeader_1x06_P2.54mm_Vertical, B.Cu at (131.3, 84.6)
- added JP1: EN, Jumper:SolderJumper-2_P1.3mm_Open_RoundedPad1.0x1.5mm, B.Cu at (183.9, 75.3)
- added P10: SMA, Connector_Coaxial:SMA_Molex_73251-1153_EdgeMount_Horizontal, B.Cu at (69.8, 72.2)
- added P11: SMA, Connector_Coaxial:SMA_Molex_73251-1153_EdgeMount_Horizontal, F.Cu at (195.3, 58.6)
- added P12: SMA, Connector_Coaxial:SMA_Molex_73251-1153_EdgeMount_Horizontal, F.Cu at (44.8, 49.3)
- added P13: SMA, Connector_Coaxial:SMA_Molex_73251-1153_EdgeMount_Horizontal, B.Cu at (195.4, 72.5)
- added P14: SMA, Connector_Coaxial:SMA_Molex_73251-1153_EdgeMount_Horizontal, B.Cu at (30.9, 49.3)
- added P3: SMA, Connector_Coaxial:SMA_Molex_73251-1153_EdgeMount_Horizontal, F.Cu at (108.7, 58.7)
- added P4: SMA, Connector_Coaxial:SMA_Molex_73251-1153_EdgeMount_Horizontal, F.Cu at (140.4, 58.7)
- added P5: SMA, Connector_Coaxial:SMA_Molex_73251-1153_EdgeMount_Horizontal, B.Cu at (108.7, 72.5)
- added P6: SMA, Connector_Coaxial:SMA_Molex_73251-1153_EdgeMount_Horizontal, B.Cu at (140.4, 72.5)
- added P7: SMA, Connector_Coaxial:SMA_Molex_73251-1153_EdgeMount_Horizontal, F.Cu at (179.3, 58.7)
- added P8: SMA, Connector_Coaxial:SMA_Molex_73251-1153_EdgeMount_Horizontal, B.Cu at (179.3, 72.5)
- added P9: SMA, Connector_Coaxial:SMA_Molex_73251-1153_EdgeMount_Horizontal, F.Cu at (69.8, 58.3)
- added U$22: , EYESPI_MINI_LOGO, F.Cu at (59.1, 85.2)
- added U9: TXS0101DBV, Package_SO:VSSOP-8_2.3x2mm_P0.5mm, B.Cu at (184.6, 77.8)
- C11, C27, C29, C30, C55, C56, C57, C61, C62, C63, C80, C83, C87, C89, C9, FL2, JP9, L17, L18, L19, L2, L23, L24, L25, L29, L30, L31, L4, L6, L8, R19, SW3, U6: moved to B.Cu
- C13: value 100p -> 100pF; moved to B.Cu
- C15: value 10n -> 10nF; moved to B.Cu
- C17: value 56p -> 100pF; moved to B.Cu
- C19: value 39p -> 82pF; moved to B.Cu
- C21: value 2.2p -> 12pF; moved to B.Cu
- C23: value 1nF -> 12pF; moved to B.Cu
- C25: value 6.2p -> 15pF; moved to B.Cu
- C54, C6: footprint Capacitor_SMD:C_0603_1608Metric -> Capacitor_SMD:C_0402_1005Metric
- C7: value 2.2pF -> 12pF; moved to B.Cu
- C76: value 1.8pF -> 3pF
- C77: value 27pF -> 6.8pF
- C78: value 1.8pF -> 1nF
- C79: value 100pH -> 100pF
- C82: value 33pF -> 220pF; moved to B.Cu
- C84: value 0.1uF -> 1uF; moved to B.Cu
- C85: value 33pF -> 270pF; moved to B.Cu
- C88: value 27pF -> 100pF; moved to B.Cu
- C90: value 1.8pF -> 47pF; moved to B.Cu
- C91: value 27pF -> 47pF; moved to B.Cu
- C92: value 1.8pF -> 18pF; moved to B.Cu
- C93: value 100pH -> 220pF; moved to B.Cu
- J4: value Conn_01x08_Pin -> RF Switch; footprint Connector_JST:JST_EH_B8B-EH-A_1x08_P2.50mm_Vertical -> Connector_PinHeader_2.54mm:PinHeader_1x05_P2.54mm_Vertical; moved to B.Cu
- JP3: value Driver -> EN; footprint Jumper:SolderJumper-3_P1.3mm_Bridged12_RoundedPad1.0x1.5mm_NumberLabels -> Jumper:SolderJumper-2_P1.3mm_Open_RoundedPad1.0x1.5mm
- L10: value 220n -> 220nH; moved to B.Cu
- L12: value 15n -> 18nH; moved to B.Cu
- L14: value 43n -> 100nH; moved to B.Cu
- L16: value 22n -> 68nH; moved to B.Cu
- L34: footprint Inductor_SMD:L_0402_1005Metric -> capstone-project:0908SQ23NGLC
- L35: value 2.2nH -> 2.4nH
- L36: value 10nH -> 150nH; moved to B.Cu
- L37: value 20nH -> 56nH; moved to B.Cu
- L38: value 23nH -> 1uH; footprint Inductor_SMD:L_0402_1005Metric -> capstone-project:IND_IMSC1008AZER_VIS; moved to B.Cu
- L39: renamed from C81; value 10pF -> 68nH; footprint Capacitor_SMD:C_0402_1005Metric -> Inductor_SMD:L_0402_1005Metric; moved to B.Cu
- L86: value 2.2nH -> 9.1nH; moved to B.Cu
- R11: value 18 -> 22; moved to B.Cu
- R14: value 1.96k -> 1.27k
- R15: value 6.04k -> 3.0k
- R17: value 1.96k -> 1.27k; moved to B.Cu
- R18: value 6.04k -> 3.0k; moved to B.Cu
- R7: value 330k -> 350; footprint Resistor_SMD:R_0603_1608Metric -> Resistor_SMD:R_0402_1005Metric; moved to B.Cu
- SW5: value SW_Push -> SKY13330-397LF; footprint Button_Switch_SMD:SW_SPST_EVQP2_MiddlePushTravel_H2.5mm -> capstone-project:SKY13330-397LF
- TP1, TP22, TP3, TP4, TP5, TP6, TP7: moved to F.Cu
- U4: footprint Package_TO_SOT_SMD:SOT-23-6 -> Package_SO:VSSOP-8_2.3x2mm_P0.5mm
- moved H5 249.6 mm to (21.8, 49.2), turned to -90 degrees
- moved H2 248.1 mm to (21.8, 81.2), turned to -90 degrees
- moved TP9 238.4 mm to (24.4, 65.3), turned to -90 degrees
- moved TP11 237.8 mm to (21.2, 75.5), turned to -90 degrees
- moved TP2 237.5 mm to (29.3, 80.8), turned to 180 degrees
- moved TP8 236.5 mm to (30.2, 83.1), turned to -90 degrees
- moved C48 235.3 mm to (21.8, 72.6), turned to -45 degrees
- moved C41 233.1 mm to (27.9, 77.1), turned to -135 degrees
- moved R12 232.0 mm to (25.5, 73.1), turned to 45 degrees
- moved C43 231.9 mm to (26.4, 74.0), turned to -135 degrees
- moved X5 231.8 mm to (23.0, 70.0), turned to -135 degrees
- moved C46 231.7 mm to (21.4, 67.4), turned to 45 degrees
- moved C42 231.6 mm to (28.8, 77.9), turned to -135 degrees
- moved TP10 229.8 mm to (21.2, 64.8), turned to -90 degrees
- moved TP5 229.5 mm to (35.3, 83.2), turned to 180 degrees
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Connections:
- C26 pad 2: /RF Subsystem/RF Frontend/UHF 6W PA/RF_{IN} -> Net-(P9-In)
- C27 pad 2: /RF Subsystem/RF Frontend/VHF 6W PA/RF_{IN} -> Net-(P10-In)
- C29 pad 1: /RF Subsystem/RF Frontend/RX_{VHF} -> /RF Subsystem/RF Frontend/TX_{VHF}
- C30 pad 1: /RF Subsystem/RF Frontend/TX_{VHF} -> /RF Subsystem/RF Frontend/RX_{VHF}
- C31 pad 1: /RF Subsystem/RF Frontend/RX_{UHF} -> /RF Subsystem/RF Frontend/TX_{UHF}
- C32 pad 1: /RF Subsystem/RF Frontend/TX_{UHF} -> /RF Subsystem/RF Frontend/RX_{UHF}
- C38 pad 2: Net-(SW3-RF1_COM) -> Net-(SW5-RF1_COM)
- C6 pad 1: /RF Subsystem/RF Frontend/RX_{UHF} -> Net-(P12-In)
- C67 pad 1: /RF Subsystem/RF Frontend/~{SW_TRX} -> /RF Subsystem/RF Frontend/UHF 6W PA/V_{EN1}
- C7 pad 1: /RF Subsystem/RF Frontend/RX_{VHF} -> Net-(P14-In)
- C70 pad 1: /RF Subsystem/RF Frontend/~{SW_TRX} -> /RF Subsystem/RF Frontend/UHF 6W PA/V_{EN2}
- C77 pad 1: Net-(C74-Pad1) -> Net-(C72-Pad1)
- C78 pad 1: Net-(C74-Pad1) -> Net-(SW3-RF1_COM)
- C78 pad 2: GND -> Net-(SW5-RF2)
- C80 pad 1: /RF Subsystem/RF Frontend/~{SW_TRX} -> /RF Subsystem/RF Frontend/VHF 6W PA/V_{EN1}
- C82 pad 1: Net-(C81-Pad2) -> Net-(C82-Pad1)
- C83 pad 1: /RF Subsystem/RF Frontend/~{SW_TRX} -> /RF Subsystem/RF Frontend/VHF 6W PA/V_{EN2}
- C88 pad 1: Net-(C88-Pad1) -> Net-(C85-Pad1)
- C90 pad 1: Net-(C88-Pad1) -> Net-(C90-Pad1)
- C91 pad 1: Net-(C88-Pad1) -> Net-(C90-Pad1)
- C92 pad 1: Net-(C88-Pad1) -> Net-(C90-Pad1)
- C93 pad 1: Net-(C88-Pad1) -> Net-(C90-Pad1)
- FL1 pad 3: /RF Subsystem/RF Frontend/TX_{UHF} -> Net-(FL1-OUT)
- FL2 pad 3: /RF Subsystem/RF Frontend/TX_{VHF} -> Net-(FL2-OUT)
- J4 pad 1: /~{AMP_SD} -> GND
- J4 pad 2: GND -> /RF Subsystem/RFSW_{TRX}
- J4 pad 3: +3.3V -> /RF Subsystem/RFSW_{BAND}
- J4 pad 4: /LRCLK -> /RF Subsystem/RFSW_{EN}
- J4 pad 5: /BCLK -> +3.3V
- JP3 pad 2: Net-(JP3-C) -> Net-(JP3-B)
- L15 pad 2: /RF Subsystem/RF Frontend/UHF 6W PA/RF_{IN} -> Net-(P9-In)
- L16 pad 2: /RF Subsystem/RF Frontend/VHF 6W PA/RF_{IN} -> Net-(P10-In)
- L32 pad 1: /RF Subsystem/RF Frontend/UHF 6W PA/RF_{IN} -> Net-(C68-Pad2)
- L36 pad 1: /RF Subsystem/RF Frontend/VHF 6W PA/RF_{IN} -> Net-(C82-Pad1)
- L39 pad 2: Net-(C81-Pad2) -> Net-(C82-Pad1)
- L86 pad 2: Net-(C88-Pad1) -> Net-(C90-Pad1)
- R14 pad 1: /RF Subsystem/RF Frontend/~{SW_TRX} -> /RF Subsystem/RF Frontend/UHF 6W PA/V_{EN1}
- R14 pad 2: /RF Subsystem/RF Frontend/~{SW_TRX} -> /RF Subsystem/RF Frontend/UHF 6W PA/V_{ENABLE1}
- R15 pad 1: /RF Subsystem/RF Frontend/~{SW_TRX} -> /RF Subsystem/RF Frontend/UHF 6W PA/V_{EN2}
- R15 pad 2: /RF Subsystem/RF Frontend/~{SW_TRX} -> /RF Subsystem/RF Frontend/UHF 6W PA/V_{ENABLE2}
- R17 pad 1: /RF Subsystem/RF Frontend/~{SW_TRX} -> /RF Subsystem/RF Frontend/VHF 6W PA/V_{EN1}
- R17 pad 2: /RF Subsystem/RF Frontend/~{SW_TRX} -> /RF Subsystem/RF Frontend/VHF 6W PA/V_{ENABLE1}
- R18 pad 1: /RF Subsystem/RF Frontend/~{SW_TRX} -> /RF Subsystem/RF Frontend/VHF 6W PA/V_{EN2}
- R18 pad 2: /RF Subsystem/RF Frontend/~{SW_TRX} -> /RF Subsystem/RF Frontend/VHF 6W PA/V_{ENABLE2}
- R7 pad 1: /~{AMP_SD} -> GND
- R7 pad 2: Net-(JP7-A) -> /RF Subsystem/RF Frontend/VHF 6W PA/RF_{IN}
- SW3 pad 8: +3.3V -> /RF Subsystem/EN_{BAND}
- SW4 pad 8: +3.3V -> /RF Subsystem/EN_{BAND}
- SW5 pad 2: Net-(R32-Pad1) -> Net-(SW5-RF1_COM)
- TP9 pad 1: /RF Subsystem/RFSW_{TRX} -> /RF Subsystem/PA_{SHUTDOWN}
- U2 pad 3: /RF Subsystem/RFSW_{TRX} -> /RF Subsystem/PA_{SHUTDOWN}
- U3 pad 3: +3.3V -> Net-(JP3-B)
- U4 pad 1: +2.5V -> /RF Subsystem/RFSW_{BAND}
- U4 pad 3: /RF Subsystem/SW_TRX -> +2.5V
- U4 pad 4: /RF Subsystem/RFSW_{TRX} -> /RF Subsystem/SW_BAND
- U4 pad 5: +2.5V -> /RF Subsystem/SW_TRX
- U4 pad 6: +3.3V -> +2.5V
- U5 pad 1: /RF Subsystem/PA_{SHUTDOWN} -> /RF Subsystem/RF Frontend/UHF 6W PA/V_{SHUTDOWN}
- U5 pad 15: /RF Subsystem/RF Frontend/~{SW_TRX} -> /RF Subsystem/RF Frontend/UHF 6W PA/V_{EN2}
- U5 pad 16: /RF Subsystem/RF Frontend/~{SW_TRX} -> /RF Subsystem/RF Frontend/UHF 6W PA/V_{EN1}
- U6 pad 1: /RF Subsystem/PA_{SHUTDOWN} -> /RF Subsystem/RF Frontend/VHF 6W PA/V_{SHUTDOWN}
- U6 pad 15: /RF Subsystem/RF Frontend/~{SW_TRX} -> /RF Subsystem/RF Frontend/VHF 6W PA/V_{EN2}
- U6 pad 16: /RF Subsystem/RF Frontend/~{SW_TRX} -> /RF Subsystem/RF Frontend/VHF 6W PA/V_{EN1}
- X1 pad 10: unconnected-(X1-Pad10) -> GND
- X1 pad 11: unconnected-(X1-Pad11) -> GND
- X1 pad 12: unconnected-(X1-Pad12) -> GND
- X1 pad 16: unconnected-(X1-Pad16) -> +3.3V
- X1 pad 2: unconnected-(X1-Pad2) -> +3.3V
- X1 pad 7: unconnected-(X1-Pad7) -> +3.3V
Routing:
- net /SCL: track 70.4 -> 0.00 mm, vias 3 -> 0
- net +3.3V: track 228.7 -> 162.6 mm, vias 7 -> 20
- net /MCU/HSPI_CS: track 57.6 -> 0.00 mm, vias 2 -> 0
- net /SDA: track 55.6 -> 0.00 mm, vias 3 -> 0
- net /MCU/VSPI_MOSI: track 49.0 -> 0.00 mm, vias 1 -> 0
- net Net-(R32-Pad1): track 48.0 -> 0.00 mm
- net /RF Subsystem/EN_{BAND}: track 0.00 -> 47.1 mm, vias 0 -> 4
- net /MCU/VSPI_MISO: track 43.8 -> 0.00 mm, vias 1 -> 0
- net /MCU/VSPI_CS: track 43.1 -> 0.00 mm, vias 1 -> 0
- net GND: track 44.6 -> 83.2 mm, vias 9 -> 676
- net /BCLK: track 36.7 -> 0.00 mm, vias 2 -> 0
- net /MCU/VSPI_SCLK: track 35.5 -> 0.00 mm, vias 1 -> 0
- net /RF Subsystem/TRX_GPIO2: track 8.19 -> 42.6 mm, vias 1 -> 2
- net /RF Subsystem/SW_BAND: track 0.00 -> 34.2 mm, vias 0 -> 2
- net /MCU/VSPI_GDO0: track 31.4 -> 0.00 mm, vias 1 -> 0
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- added copper zone on In2.Cu, net +3.3V
- added copper zone on In1.Cu, net GND
- added copper zone on In2.Cu, net GND
Other:
- board size 244.7 x 127.4 mm -> 182.6 x 41.8 mm
- copper layers 2 -> 4
- board text added: "0"
- board text added: "0 mm"
- board text added: "0.0091"
- board text added: "0.0152 mm"
- board text added: "0.0175 mm"
- board text added: "0.033"
- board text added: "0.0432 mm"
- board text added: "0.1270 mm / 0.1270 mm"
- board text added: "0.1999 mm"
- board text added: "0.3000 mm"
- board text added: "0.9906 mm"
- board text added: "1"
- board text added: "1.5422 mm"
- board text added: "144.2564 mm x 41.4767 mm"
- board text added: "3.61"
- board text added: "3.87"
- board text added: "3.9"
- board text added: "3V3"
- board text added: "4"
- board text added: "B.Cu"
- board text added: "B.Mask"
- board text added: "B.Paste"
- board text added: "B.Silkscreen"
- board text added: "BALUN_{H}"
- board text added: "BALUN_{L}"
- board text added: "BAND"
- board text added: "BIAS-T"
- board text added: "BOARD CHARACTERISTICS"
- board text added: "Board Thickness:"
- board text added: "Board overall dimensions:"
- board text added: "Bottom Silk Screen"
- board text added: "Bottom Solder Mask"
- board text added: "Bottom Solder Paste"
- board text added: "Castellated pads:"
- board text added: "Color"
- board text added: "Copper Finish:"
- board text added: "Copper Layer Count:"
- board text added: "DIPLEXER_{H}"
- board text added: "DIPLEXER_{L}"
- board text added: "Dielectric 1"
- board text added: "Dielectric 2"
- board text added: "Dielectric 3"
- board text added: "Dual-Band RF Transceiver"
- board text added: "EN"
- board text added: "ENIG"
- board text added: "Edge card connectors:"
- board text added: "Epsilon R"
- board text added: "Eric Mutton Fall 2025 REV A"
- board text added: "F.Cu"
- board text added: "F.Mask"
- board text added: "F.Paste"
- board text added: "F.Silkscreen"
- board text added: "FR4 natural"
- board text added: "FR408-HR"
- board text added: "GND"
- board text added: "IN_{H}"
- board text added: "IN_{L}"
- board text added: "Impedance Control:"
- board text added: "In1.Cu"
- board text added: "In2.Cu"
- board text added: "Layer Name"
- board text added: "Liquid Photo"
- board text added: "Loss Tangent"
- board text added: "MATCH_{H}"
- board text added: "MATCH_{L}"
- board text added: "Material"
- board text added: "Min hole diameter:"
- board text added: "Min track/spacing:"
- board text added: "No"
- board text added: "OUT_{H}"
- board text added: "OUT_{L}"
- board text added: "PA"
- board text added: "POWER AMPLIFIER"
- board text added: "Plated Board Edge:"
- board text added: "Purple"
- board text added: "RF 4-to-1 Switch"
- board text added: "RF INPUT"
- board text added: "RF OUTPUT"
- board text added: "RF SWITCH"
- board text added: "RF TRANSCEIVER"
- board text added: "RX_{H}"
- board text added: "RX_{L}"
- board text added: "SMOBC"
- board text added: "TRX"
- board text added: "TX_{H}"
- board text added: "TX_{L}"
- board text added: "Thickness (mm)"
- board text added: "Top Silk Screen"
- board text added: "Top Solder Mask"
- board text added: "Top Solder Paste"
- board text added: "Type"
- board text added: "Ultra-High Frequency Amplifier"
- board text added: "V_{CC1}"
- board text added: "V_{CC2}"
- board text added: "V_{CC3}"
- board text added: "V_{CC4}"
- board text added: "V_{EN1}"
- board text added: "V_{EN2}"
- board text added: "V_{EN3}"
- board text added: "V_{EN4}"
- board text added: "V_{SD}"
- board text added: "Very-High Frequency Amplifier"
- board text added: "White"
- board text added: "Yes"
- board text added: "copper"
- board text added: "core"
- board text added: "dBm"
- board text added: "prepreg"
- board text removed: "Audio Modulino"
- board text removed: "BALUN_{RX}"
- board text removed: "BMS"
- board text removed: "DIPLEXERS_{RX}"
- board text removed: "DIPLEXERS_{TX}"
- board text removed: "ESP32 Modulino"
- board text removed: "HMI Modulino"
- board text removed: "PA_{EXT}"
- board text removed: "Power Modulinos"
- board text removed: "RX/TX"
- board text removed: "USB-PD"
- board text removed: "Z MATCHING"
