File: Hardware/KiCAD/system-testbed/MCU.kicad_sch (KiCad schematic)
At the start: 9 parts, among them SW1 SW_Push, SW2 SW_Push, U8 ESP32-WROVER-E

Commit message: docs: added notes and a demo expectation contract to go over with the team
Parts:
- removed C1, C3, C4: 0.1u, Capacitor_SMD:C_0603_1608Metric, symbol Device:C
- removed C2: 10u, Capacitor_SMD:C_0603_1608Metric, symbol Device:C
- removed R1, R2: 10k, Resistor_SMD:R_0603_1608Metric, symbol Device:R
- removed SW1, SW2: SW_Push, Button_Switch_SMD:SW_SPST_EVQP2_MiddlePushTravel_H2.5mm, symbol Switch:SW_Push
- removed U8: ESP32-WROVER-E, capstone-project:ESP32-WROVER-IE, symbol capstone-project:ESP32-WROVER-E
