File: Hardware/KiCAD/mcu-modulino/testbed-mcu.kicad_pcb (KiCad board)
At the start: 2 copper layers, 69.6 x 55.9 mm, 24 parts, among them J1 Stemma QT, SW1 SW_Push, SW2 SW_Push, U1 ESP32-WROVER-E, U2 PCF8575DBR, X6 EYESPI, X7 EYESPI, X8 EYESPI, X9 EYESPI

Commit message: docs: added notes and a demo expectation contract to go over with the team
Parts:
- added H1: MountingHole1, ArduinoMountingHoles:Arduino_MountingHole, F.Cu at (108.2, 118.9)
- added H2: MountingHole2, ArduinoMountingHoles:Arduino_MountingHole, F.Cu at (57.4, 103.6)
- added H3: MountingHole3, ArduinoMountingHoles:Arduino_MountingHole, F.Cu at (108.2, 146.8)
- added H4: MountingHole4, ArduinoMountingHoles:Arduino_MountingHole, F.Cu at (56.1, 151.9)
- added U7: Digital_2, ArduinoPinSockets:Arduino_PinSocket_1x08_P2.54mm_Vertical, F.Cu at (44.4, 142.1)
- moved X6 181.5 mm to (67.1, 150.9), turned to 0 degrees
- moved X8 167.1 mm to (85.9, 150.9), turned to 0 degrees
- moved U2 162.3 mm to (54.9, 116.3)
- moved R4 150.7 mm to (97.5, 148.6)
- moved H20 140.3 mm to (83.8, 47.8)
- moved R3 139.3 mm to (83.3, 142.7), turned to 90 degrees
- moved SW2 138.1 mm to (66.0, 116.3)
- moved H19 132.4 mm to (94.5, 47.8)
- moved C4 131.0 mm to (69.3, 113.3), turned to 180 degrees
- moved U1 125.9 mm to (98.2, 134.1), turned to -90 degrees
- moved C1 124.8 mm to (72.1, 116.3), turned to -90 degrees
- moved J1 123.5 mm to (101.6, 104.6), turned to 180 degrees
- moved R1 123.3 mm to (77.2, 119.9)
- moved G*** 120.0 mm to (53.3, 77.7)
- moved R2 119.3 mm to (82.8, 116.3)
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Routing:
- net +3.3V: track 278.5 -> 0.00 mm, vias 10 -> 0
- net SCL: track 186.7 -> 0.00 mm, vias 13 -> 0
- net SDA: track 169.4 -> 0.00 mm, vias 12 -> 0
- net /AMP_SD: track 83.4 -> 0.00 mm, vias 2 -> 0
- net EN: track 70.2 -> 0.00 mm, vias 2 -> 0
- net /MCU/VSPI_GDO0: track 60.6 -> 0.00 mm, vias 2 -> 0
- net /MCU/HSPI_DC: track 55.9 -> 0.00 mm, vias 4 -> 0
- net /MCU/VSPI_MOSI: track 54.2 -> 0.00 mm, vias 2 -> 0
- net /MCU/VSPI_GDO2: track 49.4 -> 0.00 mm, vias 2 -> 0
- net /MCU/HMI_INT: track 49.0 -> 0.00 mm
- net /MCU/HSPI_CS: track 47.2 -> 0.00 mm, vias 5 -> 0
- net /MCU/VSPI_CS: track 47.0 -> 0.00 mm, vias 2 -> 0
- net /MCU/RF_INT: track 44.4 -> 0.00 mm, vias 2 -> 0
- net /TFT_BL_EN: track 40.8 -> 0.00 mm, vias 2 -> 0
- net /MCU/AUDIO_INT: track 40.2 -> 0.00 mm, vias 2 -> 0
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- removed copper zone on B.Cu, net GND
- removed copper zone on F.Cu, net GND
Other:
- board size 69.6 x 55.9 mm -> 68.6 x 53.3 mm
- board text removed: "Audio Connector"
- board text removed: "HMI Connector"
- board text removed: "I2C"
- board text removed: "Power Connector"
- board text removed: "RF Connector"
