File: Hardware/KiCAD/hmi-modulino-REV-B/audio-subsystem.kicad_sch (KiCad schematic)
At the start: 27 parts, among them J10 Conn_01x08_Pin, U7 MAX98357A

Commit message: docs: update all system schematics for project uniformity
Parts:
- added H1 (x2), H3, H4: MountHole, MountingHole:MountingHole_3.2mm_M3_ISO14580_Pad, symbol Mechanical:MountingHole_Pad
Connections:
- net GND: now also H1.1, H1.1, H3.1, H4.1
