File: Hardware/KiCAD/hmi-modulino-REV-B/keypad.kicad_sch (KiCad schematic)
At the start: 0 parts

Commit message: docs: update all system schematics for project uniformity
Parts:
- added D1:1, D1:10, D1:2, D1:3, D1:4, D2:1, D2:10, D2:2, D2:3, D2:4, D3:1, D3:10, D3:2, D3:3, D3:4, D4:1, D4:10, D4:2, D4:3, D4:4: D, Diode_SMD:D_0603_1608Metric, symbol Device:D_Small_Filled
- added J11: HW-834 Module, capstone-project:HW-834, symbol Connector:Conn_01x08_Socket
- added SW30: #, Button_Switch_SMD:SW_Push_1P1T_NO_CK_KMR2, symbol Switch:SW_Push_45deg
- added SW31: 1, Button_Switch_SMD:SW_Push_1P1T_NO_CK_KMR2, symbol Switch:SW_Push_45deg
- added SW32: 4, Button_Switch_SMD:SW_Push_1P1T_NO_CK_KMR2, symbol Switch:SW_Push_45deg
- added SW33: 7, Button_Switch_SMD:SW_Push_1P1T_NO_CK_KMR2, symbol Switch:SW_Push_45deg
- added SW34: 0, Button_Switch_SMD:SW_Push_1P1T_NO_CK_KMR2, symbol Switch:SW_Push_45deg
- added SW35: 2, Button_Switch_SMD:SW_Push_1P1T_NO_CK_KMR2, symbol Switch:SW_Push_45deg
- added SW36: 5, Button_Switch_SMD:SW_Push_1P1T_NO_CK_KMR2, symbol Switch:SW_Push_45deg
- added SW37: 8, Button_Switch_SMD:SW_Push_1P1T_NO_CK_KMR2, symbol Switch:SW_Push_45deg
- added SW38: *, Button_Switch_SMD:SW_Push_1P1T_NO_CK_KMR2, symbol Switch:SW_Push_45deg
- added SW39: 3, Button_Switch_SMD:SW_Push_1P1T_NO_CK_KMR2, symbol Switch:SW_Push_45deg
- added SW40: 6, Button_Switch_SMD:SW_Push_1P1T_NO_CK_KMR2, symbol Switch:SW_Push_45deg
- added SW41: 9, Button_Switch_SMD:SW_Push_1P1T_NO_CK_KMR2, symbol Switch:SW_Push_45deg
- added SW42, SW46: RIGHT, Button_Switch_SMD:SW_Push_1P1T_NO_CK_KMR2, symbol Switch:SW_Push_45deg
- added SW43: UP, Button_Switch_SMD:SW_Push_1P1T_NO_CK_KMR2, symbol Switch:SW_Push_45deg
- added SW44: DOWN, Button_Switch_SMD:SW_Push_1P1T_NO_CK_KMR2, symbol Switch:SW_Push_45deg
- added SW45: LEFT, Button_Switch_SMD:SW_Push_1P1T_NO_CK_KMR2, symbol Switch:SW_Push_45deg
- added SW47: MENU, Button_Switch_SMD:SW_Push_1P1T_NO_CK_KMR2, symbol Switch:SW_Push_45deg
- added SW48: EXIT, Button_Switch_SMD:SW_Push_1P1T_NO_CK_KMR2, symbol Switch:SW_Push_45deg
- added SW49: SK0, Button_Switch_SMD:SW_Push_1P1T_NO_CK_KMR2, symbol Switch:SW_Push_45deg
Connections:
- new net: D4:2.2 (A), SW34.1
- new net: D3:1.2 (A), SW33.1
- new net: D2:3.2 (A), SW40.1
- new net: D4:1.2 (A), SW30.1
- new net: D2:1.2 (A), SW32.1
- new net: D1:10.2 (A), SW46.1
- new net: D4:3.2 (A), SW38.1
- new net: D2:10.2 (A), SW47.1
- new net: D2:2.2 (A), SW36.1
- new net: D1:3.2 (A), SW39.1
- new net: D1:4.2 (A), SW42.1
- new net: D1:1.2 (A), SW31.1
- new net: D4:4.2 (A), SW45.1
- new net: D3:4.2 (A), SW44.1
- new net: D1:2.2 (A), SW35.1
- new net: D3:10.2 (A), SW48.1
- new net: D2:4.2 (A), SW43.1
- new net: D4:10.2 (A), SW49.1
- new net: D3:3.2 (A), SW41.1
- new net: D3:2.2 (A), SW37.1
- new net COL1: D1:1.1 (K), D2:1.1 (K), D3:1.1 (K), D4:1.1 (K), J11.5 (Pin_5)
- new net COL2: D1:2.1 (K), D2:2.1 (K), D3:2.1 (K), D4:2.1 (K), J11.6 (Pin_6)
- new net COL3: D1:3.1 (K), D2:3.1 (K), D3:3.1 (K), D4:3.1 (K), J11.7 (Pin_7)
- new net COL4: D1:4.1 (K), D2:4.1 (K), D3:4.1 (K), D4:4.1 (K), J11.8 (Pin_8)
- new net COL5: D1:10.1 (K), D2:10.1 (K), D3:10.1 (K), D4:10.1 (K)
- new net ROW1: J11.4 (Pin_4), SW31.2, SW35.2, SW39.2, SW42.2, SW46.2
- new net ROW2: J11.3 (Pin_3), SW32.2, SW36.2, SW40.2, SW43.2, SW47.2
- new net ROW3: J11.2 (Pin_2), SW33.2, SW37.2, SW41.2, SW44.2, SW48.2
- new net ROW4: J11.1 (Pin_1), SW30.2, SW34.2, SW38.2, SW45.2, SW49.2
- no-connect marks 0 -> 9
Other:
- note added: "Keypad Matrix Application Note: The ROW pins get pulled up by the GPIO expander, with one ROW being pulled down. The scanner relies on the COL pins being read in as a logic swing to low. Remarked as Domino Logic, a rail-to-rail logic swing occurs."
