File: Hardware/KiCAD/rf-modulino-REV-A/rf-amplifier-modulino/rf-amplifier-modulino-vhf.kicad_sch (KiCad schematic)
At the start: 86 parts, among them P1 SMA, P2 SMA, SW3 SKY13330-397LF, SW4 SKY13330-397LF, U2 CC1200RHBR, U3 LP5907MFX-2.5, U4 TXS0101DBV, X5 40 MHz

Commit message: docs: update all system schematics for project uniformity
Parts:
- renumbered C28 to C1, C37 to C10, C38 to C11, C39 to C12, C40 to C13, C41 to C14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
Other:
- sheet RF Frontend: file rf-transceiver-modulino-frontend.kicad_sch -> ../system-testbed/rf-frontend.kicad_sch
