File: Hardware/KiCAD/system-testbed-REV-A/system-testbed.kicad_sch (KiCad schematic)
At the start: 31 parts, among them J1 Stemma QT, J7 Stemma QT, J8 Stemma QT, X1 EYESPI, X11 EYESPI, X2 EYESPI, X3 EYESPI, X6 EYESPI, X7 EYESPI, X8 EYESPI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

Commit message: docs: update all system schematics for project uniformity
Parts:
- removed J7, J8: Stemma QT, Connector_JST:JST_SH_SM04B-SRSS-TB_1x04-1MP_P1.00mm_Horizontal, symbol Connector_Generic_Shielded:Conn_01x04_Shielded
- renumbered H1 to H21, H3 to H22, H4 to H23, H8 to H24
Other:
- sheet MCU: file MCU.kicad_sch -> ../mcu-modulino-REV-A/mcu-modulino-REV-A.kicad_sch
- sheet RF Subsystem: file rf-subsystem.kicad_sch -> ../rf-modulino-REV-A/rf-transceiver-modulino/rf-transceiver-modulino.kicad_sch
